File: Hardware/KiCad/moteur.kicad_sch (KiCad schematic)
At the start: 16 parts, among them J10 Conn_01x06, J9 Conn_01x06, U3 ZXBM5210-SP, U4 ZXBM5210-SP

Commit message: commit
Parts:
- removed D6: 1N4148WT, Diode_SMD:D_SOD-523, symbol Diode:1N4148WT
- removed D7: D_Zener, symbol Device:D_Zener
Connections:
- net V_BATT: now also C23.1, C24.2, R18.1, U3.2 (VM), U3.3 (VDD)
