File: Hardware/KiCad/regulateurs.kicad_sch (KiCad schematic)
At the start: 22 parts, among them IC2 MP1475DJ-LF-P, J8 Conn_01x02, SW2 Wurth 472121020311

Commit message: change
Changed lines of the file:
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@@
 	(bus
 		(pts
-			(xy 135.89 16.51) (xy 135.89 96.52)
+			(xy 135.89 12.7) (xy 135.89 92.71)
 		)
 		(stroke
@@
 	(bus
 		(pts
-			(xy 12.7 96.52) (xy 135.89 96.52)
+			(xy 12.7 92.71) (xy 135.89 92.71)
 		)
 		(stroke

Commit message: Update regulateurs.kicad_sch
Parts:
- C1: renamed from C14; value 22uF -> 22u
- C2: renamed from C15; value 0.1uF -> 0.1u
- C3: renamed from C16; value 0.1uF -> 0.1u
- C4: renamed from C18; value 22uF -> 22u
- C5: renamed from C20; value 22uF -> 22u
- L2: value 4.7uH -> 4.7u
- R2: renamed from R8; value R_Small -> 100K
- R5: renamed from R10; value 20R -> 20
- R7: renamed from R12; value R_Small -> 7K68
- renumbered C17 to C6, C19 to C7, R7 to R1, R11 to R3, R9 to R4, R13 to R6

Commit message: Robot
Parts:
- renumbered C1 to C14, C2 to C15, C3 to C16, C6 to C17, C4 to C18, C7 to C19, C5 to C20, R5 to R10, R3 to R11, R7 to R12, R6 to R13, R1 to R7, R2 to R8, R4 to R9
Changed lines of the file:
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@@
 	)
 	(junction
+		(at 99.06 67.31)
+		(diameter 0)
+		(color 0 0 0 0)
+	)
+	(junction
 		(at 243.84 81.28)
 		(diameter 0)
@@
 	)
 	(junction
+		(at 267.97 58.42)
+		(diameter 0)
+		(color 0 0 0 0)
+	)
+	(junction
 		(at 153.67 48.26)
 		(diameter 0)
@@
 	(wire
 		(pts
+			(xy 99.06 67.31) (xy 97.79 67.31)
+		)
+		(stroke
+			(width 0)
+			(type default)
+		)
+	)
+	(wire
+		(pts
 			(xy 80.01 138.43) (xy 92.71 138.43)
 		)
@@
 	(wire
 		(pts
-			(xy 100.33 67.31) (xy 97.79 67.31)
+			(xy 100.33 67.31) (xy 99.06 67.31)
 		)
 		(stroke
@@
 	(wire
 		(pts
+			(xy 267.97 58.42) (xy 269.24 58.42)
+		)
+		(stroke
+			(width 0)
+			(type default)
+		)
+	)
+	(wire
+		(pts
 			(xy 243.84 58.42) (xy 255.27 58.42)
 		)
@@
 	(wire
 		(pts
-			(xy 265.43 58.42) (xy 269.24 58.42)
+			(xy 265.43 58.42) (xy 267.97 58.42)
 		)
 		(stroke
@@
 		(on_board yes)
 		(dnp no)
-		(property "Reference" "R4"
+		(property "Reference" "R9"
 			(at 166.37 62.2299 0)
 			(effects
@@
 		(dnp no)
 		(fields_autoplaced yes)
-		(property "Reference" "R5"
+		(property "Reference" "R10"
 			(at 220.98 48.26 90)
 			(effects
@@
 		(dnp no)
 		(fields_autoplaced yes)
-		(property "Reference" "C5"
+		(property "Reference" "C20"
 			(at 257.81 59.6962 0)
 			(effects
@@
 		(on_board yes)
 		(dnp no)
-		(property "Reference" "#PWR?"
+		(property "Reference" "#PWR0140"
 			(at 57.15 67.31 0)
 			(effects
@@
 		(on_board yes)
 		(dnp no)
-		(property "Reference" "#PWR?"
+		(property "Reference" "#PWR0132"
 			(at 161.29 59.69 0)
 			(effects
@@
 		(on_board yes)
 		(dnp no)
-		(property "Reference" "#PWR?"
+		(property "Reference" "#PWR0133"
 			(at 170.18 59.69 0)
 			(effects
@@
 		(dnp no)
 		(fields_autoplaced yes)
-		(property "Reference" "C?"
+		(property "Reference" "C13"
 			(at 101.6 73.6599 0)
 			(effects
@@
 		(dnp no)
 		(fields_autoplaced yes)
-		(property "Reference" "#PWR?"
+		(property "Reference" "#PWR0137"
 			(at 255.27 69.85 0)
 			(effects
@@
 		(dnp no)
 		(fields_autoplaced yes)
-		(property "Reference" "#PWR?"
+		(property "Reference" "#PWR0138"
 			(at 269.24 62.23 0)
 			(effects
@@
 		(dnp no)
 		(fields_autoplaced yes)
-		(property "Reference" "C7"
+		(property "Reference" "C19"
 			(at 251.4663 67.31 90)
 			(effects
@@
 		(dnp no)
 		(fields_autoplaced yes)
-		(property "Reference" "C6"
+		(property "Reference" "C17"
 			(at 229.87 54.6162 0)
 			(effects
@@
 		(dnp no)
 		(fields_autoplaced yes)
-		(property "Reference" "SW?"
+		(property "Reference" "SW2"
 			(at 74.93 127 0)
 			(effects
@@
 		(on_board yes)
 		(dnp no)
-		(property "Reference" "R1"
+		(property "Reference" "R7"
 			(at 145.034 61.214 0)
 			(effects
@@
 		(dnp no)
 		(fields_autoplaced yes)
-		(property "Reference" "L?"
+		(property "Reference" "L2"
 			(at 236.22 53.34 90)
 			(effects
@@
 		(dnp no)
 		(fields_autoplaced yes)
-		(property "Reference" "PS?"
+		(property "Reference" "PS1"
 			(at 77.47 57.15 0)
 			(effects
@@
 		(on_board yes)
 		(dnp no)
-		(property "Reference" "R2"
+		(property "Reference" "R8"
 			(at 155.702 60.96 0)
 			(effects
@@
 		(dnp no)
 		(fields_autoplaced yes)
-		(property "Reference" "IC?"
+		(property "Reference" "IC2"
 			(at 203.2 45.72 0)
 			(effects
@@
 		(dnp no)
 		(fields_autoplaced yes)
-		(property "Reference" "C3"
+		(property "Reference" "C16"
 			(at 172.72 59.6962 0)
 			(effects
@@
 		(dnp no)
 		(fields_autoplaced yes)
-		(property "Reference" "R7"
+		(property "Reference" "R12"
 			(at 246.38 85.0899 0)
 			(effects
@@
 		(on_board yes)
 		(dnp no)
-		(property "Reference" "C1"
+		(property "Reference" "C14"
 			(at 163.83 49.5362 0)
 			(effects
@@
 		(dnp no)
 		(fields_autoplaced yes)
-		(property "Reference" "#PWR?"
+		(property "Reference" "#PWR0135"
 			(at 243.84 95.25 0)
 			(effects
@@
 		(dnp no)
 		(fields_autoplaced yes)
-		(property "Reference" "#PWR?"
+		(property "Reference" "#PWR026"
 			(at 105.41 143.51 0)
 			(effects
@@
 	)
 	(symbol
+		(lib_id "power:PWR_FLAG")
+		(at 267.97 58.42 180)
+		(unit 1)
+		(exclude_from_sim no)
+		(in_bom yes)
+		(on_board yes)
+		(dnp no)
+		(fields_autoplaced yes)
+		(property "Reference" "#FLG08"
+			(at 267.97 60.325 0)
+			(effects
+				(font
+					(size 1.27 1.27)
+				)
+				(hide yes)
+			)
+		)
+		(property "Value" "PWR_FLAG"
+			(at 267.97 62.7495 0)
+			(effects
+				(font
+					(size 1.27 1.27)
+				)
+			)
+		)
+		(property "Footprint" ""
+			(at 267.97 58.42 0)
+			(effects
+				(font
+					(size 1.27 1.27)
+				)
+				(hide yes)
+			)
+		)
+		(property "Datasheet" "~"
+			(at 267.97 58.42 0)
+			(effects
+				(font
+					(size 1.27 1.27)
+				)
+				(hide yes)
+			)
+		)
+		(property "Description" "Special symbol for telling ERC where power comes from"
+			(at 267.97 58.42 0)
+			(effects
+				(font
+					(size 1.27 1.27)
+				)
+				(hide yes)
+			)
+		)
+		(pin "1"
+		)
+		(instances
+			(project "Projet_Robot"
+				(path "/21a14c86-6900-4d4b-9d91-6c59051d0f41/9e9ae578-0fe2-489e-a2e9-26a89bc45f88"
+					(reference "#FLG08")
+					(unit 1)
+				)
+			)
+		)
+	)
+	(symbol
 		(lib_id "Device:C_Small")
 		(at 170.18 50.8 0)
@@
 		(on_board yes)
 		(dnp no)
-		(property "Reference" "C2"
+		(property "Reference" "C15"
 			(at 172.72 49.5362 0)
 			(effects
@@
 		(dnp no)
 		(fields_autoplaced yes)
-		(property "Reference" "#PWR?"
+		(property "Reference" "#PWR0136"
 			(at 243.84 69.85 0)
 			(effects
@@
 		(on_board yes)
 		(dnp no)
-		(property "Reference" "C?"
+		(property "Reference" "C12"
 			(at 47.752 66.548 0)
 			(effects
@@
 		(dnp no)
 		(fields_autoplaced yes)
-		(property "Reference" "#PWR?"
+		(property "Reference" "#PWR024"
 			(at 87.63 130.81 0)
 			(effects
@@
 		(dnp no)
 		(fields_autoplaced yes)
-		(property "Reference" "#PWR?"
+		(property "Reference" "#PWR0139"
 			(at 54.61 64.77 0)
 			(effects
@@
 		(dnp no)
 		(fields_autoplaced yes)
-		(property "Reference" "C4"
+		(property "Reference" "C18"
 			(at 246.38 59.6962 0)
 			(effects
@@
 		(dnp no)
 		(fields_autoplaced yes)
-		(property "Reference" "#PWR?"
+		(property "Reference" "#PWR025"
 			(at 44.45 153.67 0)
 			(effects
@@
 		(dnp no)
 		(fields_autoplaced yes)
-		(property "Reference" "R6"
+		(property "Reference" "R13"
 			(at 251.46 76.2 90)
 			(effects
@@
 		(dnp no)
 		(fields_autoplaced yes)
-		(property "Reference" "#PWR?"
+		(property "Reference" "#PWR0142"
 			(at 96.52 67.31 0)
 			(effects
@@
 		(on_board yes)
 		(dnp no)
-		(property "Reference" "#PWR?"
+		(property "Reference" "#PWR0143"
 			(at 54.61 86.36 0)
 			(effects
@@
 		(dnp no)
 		(fields_autoplaced yes)
-		(property "Reference" "#PWR?"
+		(property "Reference" "#PWR0131"
 			(at 203.2 76.2 0)
 			(effects
@@
 		(dnp no)
 		(fields_autoplaced yes)
-		(property "Reference" "#PWR?"
+		(property "Reference" "#PWR0141"
 			(at 149.86 46.99 0)
 			(effects
@@
 		(dnp no)
 		(fields_autoplaced yes)
-		(property "Reference" "R3"
+		(property "Reference" "R11"
 			(at 234.95 76.2 90)
 			(effects
@@
 	)
 	(symbol
+		(lib_id "power:PWR_FLAG")
+		(at 99.06 67.31 0)
+		(unit 1)
+		(exclude_from_sim no)
+		(in_bom yes)
+		(on_board yes)
+		(dnp no)
+		(fields_autoplaced yes)
+		(property "Reference" "#FLG09"
+			(at 99.06 65.405 0)
+			(effects
+				(font
+					(size 1.27 1.27)
+				)
+				(hide yes)
+			)
+		)
+		(property "Value" "PWR_FLAG"
+			(at 99.06 62.23 0)
+			(effects
+				(font
+					(size 1.27 1.27)
+				)
+			)
+		)
+		(property "Footprint" ""
+			(at 99.06 67.31 0)
+			(effects
+				(font
+					(size 1.27 1.27)
+				)
+				(hide yes)
+			)
+		)
+		(property "Datasheet" "~"
+			(at 99.06 67.31 0)
+			(effects
+				(font
+					(size 1.27 1.27)
+				)
+				(hide yes)
+			)
+		)
+		(property "Description" "Special symbol for telling ERC where power comes from"
+			(at 99.06 67.31 0)
+			(effects
+				(font
+					(size 1.27 1.27)
+				)
+				(hide yes)
+			)
+		)
+		(pin "1"
+		)
+		(instances
+			(project "Projet_Robot"
+				(path "/21a14c86-6900-4d4b-9d91-6c59051d0f41/9e9ae578-0fe2-489e-a2e9-26a89bc45f88"
+					(reference "#FLG09")
+					(unit 1)
+				)
+			)
+		)
+	)
+	(symbol
 		(lib_id "Connector_Generic:Conn_01x02")
 		(at 99.06 124.46 0)
@@
 		(dnp no)
 		(fields_autoplaced yes)
-		(property "Reference" "J?"
+		(property "Reference" "J8"
 			(at 101.6 124.4599 0)
 			(effects
@@
 		(dnp no)
 		(fields_autoplaced yes)
-		(property "Reference" "BT?"
+		(property "Reference" "BT1"
 			(at 48.26 141.6684 0)
 			(effects
@@
 		(dnp no)
 		(fields_autoplaced yes)
-		(property "Reference" "#PWR?"
+		(property "Reference" "#PWR0134"
 			(at 170.18 69.85 0)
 			(effects
