File: Hardware/KiCad/regulateurs.kicad_sch (KiCad schematic)
At the start: 22 parts, among them IC2 MP1475DJ-LF-P, J8 Conn_01x02, SW2 Wurth 472121020311

Commit message: c
Parts:
- C14, C15, C16, C17, C18, C19, C20: footprint (none) -> Capacitor_SMD:C_0201_0603Metric
- IC2: footprint SOT65P280X100-8N -> (none)
- R10, R11, R12, R13, R7, R8, R9: footprint (none) -> Resistor_SMD:R_0603_1608Metric
Changed lines of the file:
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@@
 			)
 		)
-		(property "Footprint" ""
+		(property "Footprint" "Resistor_SMD:R_0603_1608Metric"
 			(at 163.83 63.5 0)
 			(effects
@@
 			)
 		)
-		(property "Footprint" ""
+		(property "Footprint" "Resistor_SMD:R_0603_1608Metric"
 			(at 220.98 53.34 0)
 			(effects
@@
 			)
 		)
-		(property "Footprint" ""
+		(property "Footprint" "Capacitor_SMD:C_0201_0603Metric"
 			(at 255.27 60.96 0)
 			(effects
@@
 			)
 		)
-		(property "Footprint" ""
+		(property "Footprint" "Capacitor_SMD:C_0201_0603Metric"
 			(at 251.46 73.66 0)
 			(effects
@@
 			)
 		)
-		(property "Footprint" ""
+		(property "Footprint" "Capacitor_SMD:C_0201_0603Metric"
 			(at 227.33 55.88 0)
 			(effects
@@
 			)
 		)
-		(property "Footprint" ""
+		(property "Footprint" "Resistor_SMD:R_0603_1608Metric"
 			(at 149.86 62.23 0)
 			(effects
@@
 			)
 		)
-		(property "Footprint" ""
+		(property "Footprint" "Resistor_SMD:R_0603_1608Metric"
 			(at 153.67 62.23 0)
 			(effects
@@
 			)
 		)
-		(property "Footprint" "SOT65P280X100-8N"
+		(property "Footprint" ""
 			(at 214.63 148.26 0)
 			(effects
@@
 			)
 		)
-		(property "Footprint" ""
+		(property "Footprint" "Capacitor_SMD:C_0201_0603Metric"
 			(at 170.18 60.96 0)
 			(effects
@@
 			)
 		)
-		(property "Footprint" ""
+		(property "Footprint" "Resistor_SMD:R_0603_1608Metric"
 			(at 243.84 86.36 0)
 			(effects
@@
 			)
 		)
-		(property "Footprint" ""
+		(property "Footprint" "Capacitor_SMD:C_0201_0603Metric"
 			(at 161.29 50.8 0)
 			(effects
@@
 			)
 		)
-		(property "Footprint" ""
+		(property "Footprint" "Capacitor_SMD:C_0201_0603Metric"
 			(at 170.18 50.8 0)
 			(effects
@@
 			)
 		)
-		(property "Footprint" ""
+		(property "Footprint" "Capacitor_SMD:C_0201_0603Metric"
 			(at 243.84 60.96 0)
 			(effects
@@
 			)
 		)
-		(property "Footprint" ""
+		(property "Footprint" "Resistor_SMD:R_0603_1608Metric"
 			(at 251.46 81.28 0)
 			(effects
@@
 			)
 		)
-		(property "Footprint" ""
+		(property "Footprint" "Resistor_SMD:R_0603_1608Metric"
 			(at 234.95 81.28 0)
 			(effects

Commit message: j
Parts:
- BT1: footprint (none) -> Connector_JST:JST_XH_S2B-XH-A-1_1x02_P2.50mm_Horizontal
- IC2: footprint (none) -> Package_TO_SOT_SMD:TSOT-23
- J8: footprint (none) -> Connector_JST:JST_EH_B2B-EH-A_1x02_P2.50mm_Vertical
- L2: footprint (none) -> Resistor_SMD:R_0603_1608Metric
Changed lines of the file:
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@@
 			)
 		)
-		(property "Footprint" ""
+		(property "Footprint" "Resistor_SMD:R_0603_1608Metric"
 			(at 236.22 58.42 0)
 			(effects
@@
 			)
 		)
-		(property "Footprint" ""
+		(property "Footprint" "Package_TO_SOT_SMD:TSOT-23"
 			(at 214.63 148.26 0)
 			(effects
@@
 			)
 		)
-		(property "Footprint" ""
+		(property "Footprint" "Connector_JST:JST_EH_B2B-EH-A_1x02_P2.50mm_Vertical"
 			(at 99.06 124.46 0)
 			(effects
@@
 			)
 		)
-		(property "Footprint" ""
+		(property "Footprint" "Connector_JST:JST_XH_S2B-XH-A-1_1x02_P2.50mm_Horizontal"
 			(at 44.45 143.256 90)
 			(effects

Commit message: P
Connections:
- net V_BATT renamed +VBAT
Changed lines of the file:
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@@
 	)
 	(junction
+		(at 97.79 138.43)
+		(diameter 0)
+		(color 0 0 0 0)
+	)
+	(junction
 		(at 149.86 48.26)
 		(diameter 0)
@@
 	(wire
 		(pts
-			(xy 80.01 138.43) (xy 92.71 138.43)
+			(xy 80.01 138.43) (xy 97.79 138.43)
 		)
 		(stroke
@@
 	(wire
 		(pts
-			(xy 92.71 138.43) (xy 92.71 139.7)
+			(xy 54.61 78.74) (xy 54.61 72.39)
 		)
 		(stroke
@@
 	(wire
 		(pts
-			(xy 54.61 78.74) (xy 54.61 72.39)
+			(xy 255.27 58.42) (xy 265.43 58.42)
 		)
 		(stroke
@@
 	(wire
 		(pts
-			(xy 255.27 58.42) (xy 265.43 58.42)
+			(xy 163.83 58.42) (xy 170.18 58.42)
 		)
 		(stroke
@@
 	(wire
 		(pts
-			(xy 163.83 58.42) (xy 170.18 58.42)
+			(xy 97.79 138.43) (xy 105.41 138.43)
 		)
 		(stroke
@@
 	(wire
 		(pts
-			(xy 92.71 139.7) (xy 105.41 139.7)
-		)
-		(stroke
-			(width 0)
-			(type default)
-		)
-	)
-	(wire
-		(pts
 			(xy 54.61 80.01) (xy 54.61 78.74)
 		)
@@
 	)
 	(symbol
+		(lib_id "power:PWR_FLAG")
+		(at 97.79 138.43 0)
+		(unit 1)
+		(exclude_from_sim no)
+		(in_bom yes)
+		(on_board yes)
+		(dnp no)
+		(fields_autoplaced yes)
+		(property "Reference" "#FLG01"
+			(at 97.79 136.525 0)
+			(effects
+				(font
+					(size 1.27 1.27)
+				)
+				(hide yes)
+			)
+		)
+		(property "Value" "PWR_FLAG"
+			(at 97.79 133.35 0)
+			(effects
+				(font
+					(size 1.27 1.27)
+				)
+			)
+		)
+		(property "Footprint" ""
+			(at 97.79 138.43 0)
+			(effects
+				(font
+					(size 1.27 1.27)
+				)
+				(hide yes)
+			)
+		)
+		(property "Datasheet" "~"
+			(at 97.79 138.43 0)
+			(effects
+				(font
+					(size 1.27 1.27)
+				)
+				(hide yes)
+			)
+		)
+		(property "Description" "Special symbol for telling ERC where power comes from"
+			(at 97.79 138.43 0)
+			(effects
+				(font
+					(size 1.27 1.27)
+				)
+				(hide yes)
+			)
+		)
+		(pin "1"
+		)
+		(instances
+			(project ""
+				(path "/21a14c86-6900-4d4b-9d91-6c59051d0f41/9e9ae578-0fe2-489e-a2e9-26a89bc45f88"
+					(reference "#FLG01")
+					(unit 1)
+				)
+			)
+		)
+	)
+	(symbol
 		(lib_id "power:GND")
 		(at 63.5 67.31 270)
@@
 	(symbol
 		(lib_id "power:+10V")
-		(at 105.41 139.7 0)
+		(at 105.41 138.43 0)
 		(unit 1)
 		(exclude_from_sim no)
@@
 		(fields_autoplaced yes)
 		(property "Reference" "#PWR026"
-			(at 105.41 143.51 0)
+			(at 105.41 142.24 0)
 			(effects
 				(font
@@
 			)
 		)
-		(property "Value" "V_BATT"
-			(at 105.41 134.62 0)
+		(property "Value" "+VBAT"
+			(at 105.41 133.35 0)
 			(effects
 				(font
@@
 		)
 		(property "Footprint" ""
-			(at 105.41 139.7 0)
+			(at 105.41 138.43 0)
 			(effects
 				(font
@@
 		)
 		(property "Datasheet" ""
-			(at 105.41 139.7 0)
+			(at 105.41 138.43 0)
 			(effects
 				(font
@@
 		)
 		(property "Description" "Power symbol creates a global label with name \"+10V\""
-			(at 105.41 139.7 0)
+			(at 105.41 138.43 0)
 			(effects
 				(font
@@
 			)
 		)
-		(property "Value" "V_BATT"
-			(at 152.4 41.9099 0)
+		(property "Value" "+VBAT"
+			(at 149.86 38.1 0)
 			(effects
 				(font
 					(size 1.27 1.27)
 				)
-				(justify left)
 			)
 		)

Commit message: s
s
Parts:
- L2: footprint Resistor_SMD:R_0603_1608Metric -> Inductor_SMD:L_APV_ANR5040
- PS1: footprint adx:SOT95P280X125-5N -> Package_SO:TSOP-5_1.65x3.05mm_P0.95mm
Changed lines of the file:
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@@
 			)
 		)
-		(property "Footprint" "Resistor_SMD:R_0603_1608Metric"
+		(property "Footprint" "Inductor_SMD:L_APV_ANR5040"
 			(at 236.22 58.42 0)
 			(effects
@@
 			)
 		)
-		(property "Footprint" "adx:SOT95P280X125-5N"
+		(property "Footprint" "Package_SO:TSOP-5_1.65x3.05mm_P0.95mm"
 			(at 87.63 159.69 0)
 			(effects

Commit message: w
Parts:
- renumbered J8 to alim_batt, SW2 to batterie
Changed lines of the file:
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@@
 		(dnp no)
 		(fields_autoplaced yes)
-		(property "Reference" "SW2"
+		(property "Reference" "batterie"
 			(at 74.93 127 0)
 			(effects
@@
 			(project "Projet_Robot"
 				(path "/21a14c86-6900-4d4b-9d91-6c59051d0f41/9e9ae578-0fe2-489e-a2e9-26a89bc45f88"
-					(reference "SW2")
+					(reference "batterie")
 					(unit 1)
 				)
@@
 		(dnp no)
 		(fields_autoplaced yes)
-		(property "Reference" "J8"
+		(property "Reference" "alim_batt"
 			(at 101.6 124.4599 0)
 			(effects
@@
 			(project "Projet_Robot"
 				(path "/21a14c86-6900-4d4b-9d91-6c59051d0f41/9e9ae578-0fe2-489e-a2e9-26a89bc45f88"
-					(reference "J8")
-					(unit 1)
-				)
+					(reference "alim_batt")
+					(unit 1)
+				)

Commit message: s
Parts:
- renumbered alim_batt to alim_batt1, batterie to batterie1
Changed lines of the file:
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@@
 		(dnp no)
 		(fields_autoplaced yes)
-		(property "Reference" "batterie"
+		(property "Reference" "batterie1"
 			(at 74.93 127 0)
 			(effects
@@
 			(project "Projet_Robot"
 				(path "/21a14c86-6900-4d4b-9d91-6c59051d0f41/9e9ae578-0fe2-489e-a2e9-26a89bc45f88"
-					(reference "batterie")
+					(reference "batterie1")
 					(unit 1)
 				)
@@
 		(dnp no)
 		(fields_autoplaced yes)
-		(property "Reference" "alim_batt"
+		(property "Reference" "alim_batt1"
 			(at 101.6 124.4599 0)
 			(effects
@@
 			(project "Projet_Robot"
 				(path "/21a14c86-6900-4d4b-9d91-6c59051d0f41/9e9ae578-0fe2-489e-a2e9-26a89bc45f88"
-					(reference "alim_batt")
-					(unit 1)
-				)
+					(reference "alim_batt1")
+					(unit 1)
+				)

Commit message: q
Parts:
- IC2: footprint Package_TO_SOT_SMD:TSOT-23 -> Package_TO_SOT_SMD:TSOT-23-8_HandSoldering
Changed lines of the file:
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@@
 			)
 		)
-		(property "Footprint" "Package_TO_SOT_SMD:TSOT-23"
+		(property "Footprint" "Package_TO_SOT_SMD:TSOT-23-8_HandSoldering"
 			(at 214.63 148.26 0)
 			(effects

Commit message: s
Other:
- moved on the sheet: C13
Changed lines of the file:
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@@
 	(symbol
 		(lib_id "Device:C")
-		(at 97.79 74.93 180)
+		(at 97.79 74.93 0)
+		(mirror x)
 		(unit 1)
 		(exclude_from_sim no)
@@
 		(on_board yes)
 		(dnp no)
-		(fields_autoplaced yes)
 		(property "Reference" "C13"
-			(at 101.6 73.6599 0)
+			(at 93.98 73.6599 0)
 			(effects
 				(font
@@
 		)
 		(property "Value" "1u"
-			(at 101.6 76.1999 0)
+			(at 93.98 76.1999 0)
 			(effects
 				(font
@@
 		)
 		(property "Footprint" "Capacitor_SMD:C_0603_1608Metric"
-			(at 96.8248 71.12 0)
+			(at 98.7552 71.12 0)
 			(effects
 				(font
