File: Hardware/KiCad/regulateurs.kicad_sch (KiCad schematic)
At the start: 22 parts, among them IC2 MP1475DJ-LF-P

Commit message: s
Parts:
- R10: value 20 -> 20k
Changed lines of the file:
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@@
 			)
 		)
-		(property "Value" "20"
+		(property "Value" "20k"
 			(at 220.98 50.8 90)
 			(effects

Commit message: s
Parts:
- removed batterie1: Wurth 472121020311, Button_Switch_SMD:Nidec_Copal_CAS-120A, symbol Switch:SW_Nidec_CAS-120A1
- added S1: 1101M2S3CQE2, KiCad:1101M2S3QE2, symbol 1101M2S3CQE2:1101M2S3CQE2
- BT1: now left out of the parts list
- C14, C18, C20: footprint Capacitor_SMD:C_0201_0603Metric -> Capacitor_SMD:C_0805_2012Metric
- C15, C16: value 0.1u -> 100n; footprint Capacitor_SMD:C_0201_0603Metric -> Capacitor_SMD:C_0402_1005Metric
- C17: value 0.1uF -> 100n; footprint Capacitor_SMD:C_0201_0603Metric -> Capacitor_SMD:C_0402_1005Metric
- C19: value 15pF -> 15p; footprint Capacitor_SMD:C_0201_0603Metric -> Capacitor_SMD:C_0402_1005Metric
- J1: renamed from alim_batt1; value Conn_01x02 -> Conn_Battery_Cell
- L2: value 4.7u -> 4u7
- R13: value 40.2K -> 40k2
Connections:
- net +VBAT: now also S1.2
- net at BT1.1 (+): now also J1.2 (Pin_2), S1.3
- no-connect marks 0 -> 1

Commit message: sss
Changed lines of the file:
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@@
 		(lib_id "Device:R_Small")
 		(at 149.86 62.23 0)
+		(mirror y)
 		(unit 1)
 		(exclude_from_sim no)
@@
 		(dnp no)
 		(property "Reference" "R7"
-			(at 145.034 61.214 0)
+			(at 154.686 61.214 0)
 			(effects
 				(font
@@
 		)
 		(property "Value" "100K"
-			(at 142.748 63.754 0)
+			(at 156.972 63.754 0)
 			(effects
 				(font

Commit message: R
Changed lines of the file:
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@@
 		(lib_id "Device:C_Small")
 		(at 170.18 50.8 0)
+		(mirror y)
 		(unit 1)
 		(exclude_from_sim no)
@@
 		(dnp no)
 		(property "Reference" "C15"
-			(at 172.72 49.5362 0)
+			(at 167.64 49.5362 0)
 			(effects
 				(font
@@
 		)
 		(property "Value" "100n"
-			(at 172.72 52.578 0)
+			(at 167.64 52.578 0)
 			(effects
 				(font

Commit message: check LF
Parts:
- removed R8: 100K, Resistor_SMD:R_0603_1608Metric, symbol Device:R_Small
Connections:
- net SW: now reaches C17.2, IC2.3 (SW), L2.1
Changed lines of the file:
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@@
-	)
-	(junction
-		(at 153.67 76.2)
-		(diameter 0)
-		(color 0 0 0 0)
 	)
 	(junction
@@
 		(color 0 0 0 0)
 	)
-	(junction
-		(at 153.67 48.26)
-		(diameter 0)
-		(color 0 0 0 0)
-	)
 	(no_connect
 		(at 80.01 133.35)
@@
 	(wire
 		(pts
-			(xy 153.67 76.2) (xy 187.96 76.2)
-		)
-		(stroke
-			(width 0)
-			(type default)
-		)
-	)
-	(wire
-		(pts
 			(xy 187.96 52.07) (xy 184.15 52.07)
 		)
@@
 	(wire
 		(pts
-			(xy 153.67 64.77) (xy 153.67 76.2)
-		)
-		(stroke
-			(width 0)
-			(type default)
-		)
-	)
-	(wire
-		(pts
 			(xy 187.96 63.5) (xy 187.96 76.2)
 		)
@@
 	(wire
 		(pts
-			(xy 149.86 48.26) (xy 153.67 48.26)
+			(xy 149.86 48.26) (xy 161.29 48.26)
 		)
 		(stroke
@@
 	(wire
 		(pts
-			(xy 153.67 48.26) (xy 153.67 59.69)
-		)
-		(stroke
-			(width 0)
-			(type default)
-		)
-	)
-	(wire
-		(pts
 			(xy 91.44 67.31) (xy 97.79 67.31)
 		)
@@
 	(wire
 		(pts
-			(xy 149.86 76.2) (xy 153.67 76.2)
+			(xy 149.86 76.2) (xy 187.96 76.2)
 		)
 		(stroke
@@
 	(wire
 		(pts
-			(xy 153.67 48.26) (xy 161.29 48.26)
-		)
-		(stroke
-			(width 0)
-			(type default)
-		)
-	)
-	(wire
-		(pts
 			(xy 163.83 60.96) (xy 163.83 58.42)
 		)
@@
 			(width 0)
 			(type default)
+		)
+	)
+	(label "SW"
+		(at 218.44 58.42 0)
+		(effects
+			(font
+				(size 1.27 1.27)
+			)
+			(justify left bottom)
 		)
 	)
@@
 					(unit 1)
 				)
-			)
-		)
-	)
-	(symbol
-		(lib_id "Device:R_Small")
-		(at 153.67 62.23 0)
-		(unit 1)
-		(exclude_from_sim no)
-		(in_bom yes)
-		(on_board yes)
-		(dnp no)
-		(property "Reference" "R8"
-			(at 155.702 60.96 0)
-			(effects
-				(font
-					(size 1.016 1.016)
-				)
-				(justify left)
-			)
-		)
-		(property "Value" "100K"
-			(at 155.448 63.754 0)
-			(effects
-				(font
-					(size 1.27 1.27)
-				)
-				(justify left)
-			)
-		)
-		(property "Footprint" "Resistor_SMD:R_0603_1608Metric"
-			(at 153.67 62.23 0)
-			(effects
-				(font
-					(size 1.27 1.27)
-				)
-				(hide yes)
-			)
-		)
-		(property "Datasheet" "~"
-			(at 153.67 62.23 0)
-			(effects
-				(font
-					(size 1.27 1.27)
-				)
-				(hide yes)
-			)
-		)
-		(property "Description" "Resistor, small symbol"
-			(at 153.67 62.23 0)
-			(effects
-				(font
-					(size 1.27 1.27)
-				)
-				(hide yes)
-			)
-		)
-		(pin "2"
-		)
-		(pin "1"
-		)
-		(instances
-			(project ""
-				(path "/21a14c86-6900-4d4b-9d91-6c59051d0f41/9e9ae578-0fe2-489e-a2e9-26a89bc45f88"
-					(reference "R8")
-					(unit 1)
-				)
-			)
-			(project ""
-				(path "/93119413-89cd-4eb7-94e5-66a9033edb4e/5b707b38-31ab-4d40-af5c-5c07b9e7f3b7"
-					(reference "R6")
-					(unit 1)
-				)
-			)
-			(project ""
-				(path "/bd05b7a9-402f-4660-98a3-5b54bc637b02/e2d0a223-2588-4552-8b74-bae61965aad2"
-					(reference "R10")
-					(unit 1)
-				)
-			)
-			(project "regulateurs"
-				(path "/f59dd815-4ba9-415e-b839-e2d0d5228d08"
-					(reference "R2")
-					(unit 1)
-				)
