File: Hardware/KiCad/µcontrolleur.kicad_sch (KiCad schematic)
At the start: 22 parts, among them J1 Conn_02x07_Odd_Even, SW1 SW_Push, U1 STM32G431CBUx, Y1 16MHz

Commit message: commit
Parts:
- removed J1: Conn_02x07_Odd_Even, Connector_PinHeader_1.27mm:PinHeader_2x07_P1.27mm_Vertical_SMD, symbol Connector_Generic:Conn_02x07_Odd_Even
- removed JP1, JP2: SolderJumper_2_Open, Jumper:SolderJumper-2_P1.3mm_Open_TrianglePad1.0x1.5mm, symbol Jumper:SolderJumper_2_Open
- added J11: Conn_ST_STDC14, symbol Connector:Conn_ST_STDC14
Connections:
- net TIM2_CH2 is gone; now on net TIM2_CH1: U1.9 (PA1)
- net +3.3V: now also J11.3 (VCC)
- net GND: now also J11.5 (GND), J11.7 (GND)
- net NRST: now also J11.12 (~{RST})
- net STATUS_LED: now also U1.4 (PC15); no longer U1.17 (PB0)
- net SWCLK: now also J11.6 (JCLK/SWCLK)
- net SWDIO: now also J11.4 (JTMS/SWDIO)
- net VCP_RX: now also J11.13 (VCP_RX)
- net VCP_TX: now also J11.14 (VCP_TX)
- net LIDAR_USART2_TX: now reaches U1.10 (PA2)
- no-connect marks 27 -> 25

Commit message: change
Changed lines of the file:
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@@
 	)
 	(junction
-		(at 87.63 68.58)
+		(at 87.63 69.85)
 		(diameter 0)
 		(color 0 0 0 0)
@@
 	)
 	(junction
-		(at 88.9 46.99)
+		(at 90.17 46.99)
 		(diameter 0)
 		(color 0 0 0 0)
@@
 	(wire
 		(pts
-			(xy 87.63 68.58) (xy 87.63 46.99)
+			(xy 90.17 46.99) (xy 90.17 69.85)
 		)
 		(stroke
@@
 	(wire
 		(pts
-			(xy 87.63 46.99) (xy 88.9 46.99)
-		)
-		(stroke
-			(width 0)
-			(type default)
-		)
-	)
-	(wire
-		(pts
 			(xy 222.25 64.77) (xy 226.06 64.77)
 		)
@@
 	(wire
 		(pts
-			(xy 87.63 72.39) (xy 87.63 68.58)
+			(xy 87.63 72.39) (xy 87.63 69.85)
 		)
 		(stroke
@@
 	(wire
 		(pts
-			(xy 88.9 46.99) (xy 99.06 46.99)
+			(xy 90.17 46.99) (xy 99.06 46.99)
 		)
 		(stroke
@@
 	(wire
 		(pts
+			(xy 90.17 69.85) (xy 87.63 69.85)
+		)
+		(stroke
+			(width 0)
+			(type default)
+		)
+	)
+	(wire
+		(pts
 			(xy 62.23 97.79) (xy 62.23 110.49)
 		)
@@
 	(wire
 		(pts
-			(xy 223.52 110.49) (xy 234.95 110.49)
+			(xy 87.63 69.85) (xy 87.63 67.31)
+		)
+		(stroke
+			(width 0)
+			(type default)
+		)
+	)
+	(wire
+		(pts
+			(xy 90.17 46.99) (xy 88.9 46.99)
 		)
 		(stroke
@@
 		(pts
 			(xy 100.33 100.33) (xy 116.84 100.33)
+		)
+		(stroke
+			(width 0)
+			(type default)
+		)
+	)
+	(wire
+		(pts
+			(xy 219.71 110.49) (xy 234.95 110.49)
 		)
 		(stroke
@@
 	)
 	(label "NRST"
+		(at 219.71 110.49 0)
+		(effects
+			(font
+				(size 1.27 1.27)
+			)
+			(justify left bottom)
+		)
+	)
+	(label "NRST"
 		(at 25.4 73.66 0)
 		(effects
@@
 			)
 			(justify right bottom)
-		)
-	)
-	(global_label "NRST"
-		(shape input)
-		(at 223.52 110.49 180)
-		(fields_autoplaced yes)
-		(effects
-			(font
-				(size 1.27 1.27)
-			)
-			(justify right)
-		)
-		(property "Intersheetrefs" "${INTERSHEET_REFS}"
-			(at 215.7572 110.49 0)
-			(effects
-				(font
-					(size 1.27 1.27)
-				)
-				(justify right)
-				(hide yes)
-			)
 		)
 	)
@@
 	(symbol
 		(lib_id "power:PWR_FLAG")
-		(at 87.63 68.58 270)
+		(at 87.63 67.31 0)
 		(unit 1)
 		(exclude_from_sim no)
@@
 		(fields_autoplaced yes)
 		(property "Reference" "#FLG04"
-			(at 89.535 68.58 0)
+			(at 87.63 65.405 0)
 			(effects
 				(font
@@
 		)
 		(property "Value" "PWR_FLAG"
-			(at 91.44 68.5799 90)
+			(at 90.17 66.0399 0)
 			(effects
 				(font
@@
 		)
 		(property "Footprint" ""
-			(at 87.63 68.58 0)
+			(at 87.63 67.31 0)
 			(effects
 				(font
@@
 		)
 		(property "Datasheet" "~"
-			(at 87.63 68.58 0)
+			(at 87.63 67.31 0)
 			(effects
 				(font
@@
 		)
 		(property "Description" "Special symbol for telling ERC where power comes from"
-			(at 87.63 68.58 0)
-			(effects
-				(font
+			(at 87.63 67.31 0)
+			(effects
+				(font

Commit message: change
Connections:
- net TIM1_CH1 renamed PWM_Mot1_CH1
- net TIM1_CH2 renamed PWM_Mot1_CH2
- net TIM2_CH1 renamed PWM_Mot2_CH1
- net PWM_Mot2_CH1: no longer U1.9 (PA1)
- new net PWM_Mot2_CH2: U1.9 (PA1)
Changed lines of the file:
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@@
 		)
 	)
-	(hierarchical_label "TIM1_CH2"
+	(hierarchical_label "PWM_Mot2_CH1"
+		(shape input)
+		(at 107.95 92.71 0)
+		(effects
+			(font
+				(size 1.27 1.27)
+			)
+			(justify left)
+		)
+	)
+	(hierarchical_label "PWM_Mot2_CH2"
+		(shape input)
+		(at 115.57 82.55 0)
+		(effects
+			(font
+				(size 1.27 1.27)
+			)
+			(justify left)
+		)
+	)
+	(hierarchical_label "PWM_Mot1_CH2"
 		(shape input)
 		(at 116.84 102.87 0)
@@
 		)
 	)
-	(hierarchical_label "TIM2_CH1"
+	(hierarchical_label "ENC1_PH2"
 		(shape input)
-		(at 107.95 92.71 0)
+		(at 129.54 148.59 180)
 		(effects
 			(font
 				(size 1.27 1.27)
 			)
-			(justify left)
-		)
-	)
-	(hierarchical_label "TIM1_CH1"
-		(shape input)
-		(at 116.84 100.33 0)
-		(effects
-			(font
-				(size 1.27 1.27)
-			)
-			(justify left)
+			(justify right)
 		)
 	)
@@
 		)
 	)
-	(hierarchical_label "TIM2_CH1"
+	(hierarchical_label "ENC2_PH2"
 		(shape input)
-		(at 115.57 82.55 0)
+		(at 129.54 166.37 180)
 		(effects
 			(font
 				(size 1.27 1.27)
 			)
-			(justify left)
+			(justify right)
+		)
+	)
+	(hierarchical_label "ENC1_PH1"
+		(shape input)
+		(at 129.54 151.13 180)
+		(effects
+			(font
+				(size 1.27 1.27)
+			)
+			(justify right)
 		)
 	)
@@
 		)
 	)
+	(hierarchical_label "ENC2_PH1"
+		(shape input)
+		(at 129.54 168.91 180)
+		(effects
+			(font
+				(size 1.27 1.27)
+			)
+			(justify right)
+		)
+	)
 	(hierarchical_label "LIDAR_USART2_TX"
 		(shape input)
@@
 		)
 	)
+	(hierarchical_label "PWM_Mot1_CH1"
+		(shape input)
+		(at 116.84 100.33 0)
+		(effects
+			(font
+				(size 1.27 1.27)
+			)
+			(justify left)
+		)
+	)

Commit message: Robot
Parts:
- added D3, D4, D5: LED_Small, LED_SMD:LED_0201_0603Metric, symbol Device:LED_Small
- added R14, R5, R6: 1k, Resistor_SMD:R_0603_1608Metric, symbol Device:R
- added SW3: SW_Push, symbol Switch:SW_Push
- R3, R4: value 100k -> 1k
Connections:
- net ENC1_PH1: now also U1.33 (PA11)
- net ENC1_PH2: now also U1.34 (PA12)
- net ENC2_PH1: now also U1.12 (PA4)
- net ENC2_PH2: now also U1.17 (PB0)
- net GND: now also J11.11 (GNDDetect), R14.1, R5.1, R6.1, SW3.2
- net BOUTON_Chat/Souris: now reaches U1.28 (PB15)
- net BOUTON_Chat/Souris: now also SW3.1
- net STATUS_SOURIS_LED: now reaches U1.3 (PC14)
- net STATUS_SOURIS_LED: now also D5.2 (A)
- net STATUS_LED renamed STATUS_CHAT_LED
- net SWO: no longer names the net of U1.41 (PB3)
- new net: D3.1 (K), R5.2
- new net: D4.1 (K), R6.2
- new net: D5.1 (K), R14.2
- new net +5V: D3.2 (A)
- new net V_BATT: D4.2 (A)
- no-connect marks 25 -> 20
Other:
- note added: "Bouton Chat/Souris"
- moved on the sheet: C3, C4, D1, D2, R3, R4, SW1, Y1
