File: Hardware/KiCad/µcontrolleur.kicad_sch (KiCad schematic)
At the start: 31 parts, among them J11 Conn_ST_STDC14, SW1 SW_Push, SW3 SW_Push, U1 STM32G431CBUx, Y1 16MHz

Commit message: s
Parts:
- added C32: 100nf, Capacitor_SMD:C_0201_0603Metric, symbol Device:C
- added R17: 10k, Resistor_SMD:R_0603_1608Metric, symbol Device:R
- added R20: 10K, Resistor_SMD:R_0603_1608Metric, symbol Device:R
Connections:
- net +3.3V: now also R17.1
- net BOUTON_Chat/Souris: now also C32.1, R20.1; no longer SW3.1
- net GND: now also C32.2
- new net: R17.2, R20.2, SW3.1

Commit message: s
s
Parts:
- removed H1, H2, H3, H4: MountingHole, MountingHole:MountingHole_3.2mm_M3_Pad_Via, symbol Mechanical:MountingHole
- added H1, H2, H3, H4: MountingHole_Pad, MountingHole:MountingHole_3.2mm_M3_ISO7380_Pad, symbol Mechanical:MountingHole_Pad
Connections:
- net GND: now also H1.1, H2.1, H3.1, H4.1

Commit message: w
Parts:
- H1, H2, H3, H4: footprint MountingHole:MountingHole_3.2mm_M3_ISO7380_Pad -> MountingHole:MountingHole_3.2mm_M3_Pad_Via
- renumbered SW1 to B-Res, SW3 to ch/sou
Changed lines of the file:
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@@
 			)
 		)
-		(property "Footprint" "MountingHole:MountingHole_3.2mm_M3_ISO7380_Pad"
+		(property "Footprint" "MountingHole:MountingHole_3.2mm_M3_Pad_Via"
 			(at 87.63 182.88 0)
 			(effects
@@
 		(dnp no)
 		(fields_autoplaced yes)
-		(property "Reference" "SW1"
+		(property "Reference" "B-Res"
 			(at 256.54 100.33 0)
 			(effects
@@
 			(project ""
 				(path "/21a14c86-6900-4d4b-9d91-6c59051d0f41/31be01aa-b096-4901-8c4f-f2a7c3166097"
-					(reference "SW1")
+					(reference "B-Res")
 					(unit 1)
 				)
@@
 			)
 		)
-		(property "Footprint" "MountingHole:MountingHole_3.2mm_M3_ISO7380_Pad"
+		(property "Footprint" "MountingHole:MountingHole_3.2mm_M3_Pad_Via"
 			(at 95.25 182.88 0)
 			(effects
@@
 			)
 		)
-		(property "Footprint" "MountingHole:MountingHole_3.2mm_M3_ISO7380_Pad"
+		(property "Footprint" "MountingHole:MountingHole_3.2mm_M3_Pad_Via"
 			(at 80.01 182.88 0)
 			(effects
@@
 		(dnp no)
 		(fields_autoplaced yes)
-		(property "Reference" "SW3"
+		(property "Reference" "ch/sou"
 			(at 264.16 142.24 0)
 			(effects
@@
 			(project "Projet_Robot"
 				(path "/21a14c86-6900-4d4b-9d91-6c59051d0f41/31be01aa-b096-4901-8c4f-f2a7c3166097"
-					(reference "SW3")
+					(reference "ch/sou")
 					(unit 1)
 				)
@@
 			)
 		)
-		(property "Footprint" "MountingHole:MountingHole_3.2mm_M3_ISO7380_Pad"
+		(property "Footprint" "MountingHole:MountingHole_3.2mm_M3_Pad_Via"
 			(at 72.39 182.88 0)
 			(effects

Commit message: s
Parts:
- renumbered B-Res to B-Res1, ch/sou to ch/sou1
Changed lines of the file:
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@@
 		(dnp no)
 		(fields_autoplaced yes)
-		(property "Reference" "B-Res"
+		(property "Reference" "B-Res1"
 			(at 256.54 100.33 0)
 			(effects
@@
 			(project ""
 				(path "/21a14c86-6900-4d4b-9d91-6c59051d0f41/31be01aa-b096-4901-8c4f-f2a7c3166097"
-					(reference "B-Res")
+					(reference "B-Res1")
 					(unit 1)
 				)
@@
 		(dnp no)
 		(fields_autoplaced yes)
-		(property "Reference" "ch/sou"
+		(property "Reference" "ch/sou1"
 			(at 264.16 142.24 0)
 			(effects
@@
 			(project "Projet_Robot"
 				(path "/21a14c86-6900-4d4b-9d91-6c59051d0f41/31be01aa-b096-4901-8c4f-f2a7c3166097"
-					(reference "ch/sou")
+					(reference "ch/sou1")
 					(unit 1)
 				)

Commit message: s
Connections:
- net ENC1_PH1: now also U1.8 (PA0); no longer U1.14 (PA6)
- net ENC1_PH2: now also U1.9 (PA1); no longer U1.15 (PA7)
- net ENC2_PH1: now also U1.33 (PA11); no longer U1.17 (PB0)
- net ENC2_PH2: now also U1.34 (PA12); no longer U1.18 (PB1)
- net PWM_Mot1_CH1: now also U1.14 (PA6); no longer U1.8 (PA0)
- net PWM_Mot1_CH2: now also U1.15 (PA7); no longer U1.9 (PA1)
- net PWM_Mot2_CH1: now also U1.17 (PB0); no longer U1.33 (PA11)
- net PWM_Mot2_CH2: now also U1.18 (PB1); no longer U1.34 (PA12)
Changed lines of the file:
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@@
+		)
+	)
+	(hierarchical_label "ACC_INT1"
+		(shape input)
+		(at 59.69 151.13 180)
+		(effects
+			(font
+				(size 1.27 1.27)
+			)
+			(justify right)
+		)
+	)
+	(hierarchical_label "TOF3_XSHUT"
+		(shape input)
+		(at 57.15 105.41 180)
+		(effects
+			(font
+				(size 1.27 1.27)
+			)
+			(justify right)
+		)
+	)
+	(hierarchical_label "tof2_GPIO"
+		(shape input)
+		(at 63.5 130.81 180)
+		(effects
+			(font
+				(size 1.27 1.27)
+			)
+			(justify right)
+		)
+	)
+	(hierarchical_label "tof4_GPIO"
+		(shape input)
+		(at 63.5 135.89 180)
+		(effects
+			(font
+				(size 1.27 1.27)
+			)
+			(justify right)
+		)
+	)
+	(hierarchical_label "TOF1_XSHUT"
+		(shape input)
+		(at 105.41 118.11 0)
+		(effects
+			(font
+				(size 1.27 1.27)
+			)
+			(justify left)
+		)
+	)
+	(hierarchical_label "tof3_GPIO"
+		(shape input)
+		(at 63.5 133.35 180)
+		(effects
+			(font
+				(size 1.27 1.27)
+			)
+			(justify right)
+		)
+	)
+	(hierarchical_label "tof1_GPIO"
+		(shape input)
+		(at 63.5 128.27 180)
+		(effects
+			(font
+				(size 1.27 1.27)
+			)
+			(justify right)
+		)
+	)
+	(hierarchical_label "Bluetooth_USART3_RX"
+		(shape input)
+		(at 59.69 146.05 180)
+		(effects
+			(font
+				(size 1.27 1.27)
+			)
+			(justify right)
+		)
+	)
+	(hierarchical_label "ENC1_PH1"
+		(shape input)
+		(at 109.22 80.01 0)
+		(effects
+			(font
+				(size 1.27 1.27)
+			)
+			(justify left)
+		)
+	)
+	(hierarchical_label "PWM_Mot2_CH2"
+		(shape input)
+		(at 59.69 120.65 180)
+		(effects
+			(font
+				(size 1.27 1.27)
+			)
+			(justify right)
+		)
+	)
+	(hierarchical_label "TOF4_XSHUT"
+		(shape input)
+		(at 63.5 125.73 180)
+		(effects
+			(font
+				(size 1.27 1.27)
+			)
+			(justify right)
+		)
+	)
+	(hierarchical_label "ACC_INT2"
+		(shape input)
+		(at 59.69 148.59 180)
+		(effects
+			(font
+				(size 1.27 1.27)
+			)
+			(justify right)
+		)
+	)
+	(hierarchical_label "PWM_Mot1_CH2"
+		(shape input)
+		(at 114.3 97.79 0)
+		(effects
+			(font
+				(size 1.27 1.27)
+			)
+			(justify left)
 		)
 	)
 	(hierarchical_label "ENC2_PH1"
 		(shape input)
+		(at 109.22 107.95 0)
+		(effects
+			(font
+				(size 1.27 1.27)
+			)
+			(justify left)
+		)
+	)
+	(hierarchical_label "I2C1_SDA"
+		(shape input)
+		(at 36.83 140.97 180)
+		(effects
+			(font
+				(size 1.27 1.27)
+			)
+			(justify right)
+		)
+	)
+	(hierarchical_label "I2C1_SCL"
+		(shape input)
+		(at 31.75 138.43 180)
+		(effects
+			(font
+				(size 1.27 1.27)
+			)
+			(justify right)
+		)
+	)
+	(hierarchical_label "LIDAR_USART2_RX"
+		(shape input)
+		(at 109.22 85.09 0)
+		(effects
+			(font
+				(size 1.27 1.27)
+			)
+			(justify left)
+		)
+	)
+	(hierarchical_label "ENC2_PH2"
+		(shape input)
+		(at 109.22 110.49 0)
+		(effects
+			(font
+				(size 1.27 1.27)
+			)
+			(justify left)
+		)
+	)
+	(hierarchical_label "TOF2_XSHUT"
+		(shape input)
+		(at 57.15 102.87 180)
+		(effects
+			(font
+				(size 1.27 1.27)
+			)
+			(justify right)
+		)
+	)
+	(hierarchical_label "Bluetooth_USART3_TX"
+		(shape input)
+		(at 59.69 143.51 180)
+		(effects
+			(font
+				(size 1.27 1.27)
+			)
+			(justify right)
+		)
+	)
+	(hierarchical_label "ENC1_PH2"
+		(shape input)
+		(at 109.22 82.55 0)
+		(effects
+			(font
+				(size 1.27 1.27)
+			)
+			(justify left)
+		)
+	)
+	(hierarchical_label "M_CTR"
+		(shape input)
+		(at 114.3 100.33 0)
+		(effects
+			(font
+				(size 1.27 1.27)
+			)
+			(justify left)
+		)
+	)
+	(hierarchical_label "PWM_Mot2_CH1"
+		(shape input)
 		(at 59.69 118.11 180)
 		(effects
@@
 		)
 	)
-	(hierarchical_label "PWM_Mot2_CH2"
-		(shape input)
-		(at 109.22 110.49 0)
-		(effects
-			(font
-				(size 1.27 1.27)
-			)
-			(justify left)
-		)
-	)
-	(hierarchical_label "ENC1_PH2"
-		(shape input)
-		(at 114.3 97.79 0)
-		(effects
-			(font
-				(size 1.27 1.27)
-			)
-			(justify left)
-		)
-	)
-	(hierarchical_label "ACC_INT1"
-		(shape input)
-		(at 59.69 151.13 180)
-		(effects
-			(font
-				(size 1.27 1.27)
-			)
-			(justify right)
-		)
-	)
-	(hierarchical_label "TOF3_XSHUT"
-		(shape input)
-		(at 57.15 105.41 180)
-		(effects
-			(font
-				(size 1.27 1.27)
-			)
-			(justify right)
-		)
-	)
-	(hierarchical_label "tof2_GPIO"
-		(shape input)
-		(at 63.5 130.81 180)
-		(effects
-			(font
-				(size 1.27 1.27)
-			)
-			(justify right)
-		)
-	)
-	(hierarchical_label "tof4_GPIO"
-		(shape input)
-		(at 63.5 135.89 180)
-		(effects
-			(font
-				(size 1.27 1.27)
-			)
-			(justify right)
-		)
-	)
-	(hierarchical_label "TOF1_XSHUT"
-		(shape input)
-		(at 105.41 118.11 0)
-		(effects
-			(font
-				(size 1.27 1.27)
-			)
-			(justify left)
-		)
-	)
-	(hierarchical_label "ENC1_PH1"
+	(hierarchical_label "PWM_Mot1_CH1"
 		(shape input)
 		(at 114.3 95.25 0)
 		(effects
 			(font
-				(size 1.27 1.27)
-			)
-			(justify left)
-		)
-	)
-	(hierarchical_label "tof3_GPIO"
-		(shape input)
-		(at 63.5 133.35 180)
-		(effects
-			(font
-				(size 1.27 1.27)
-			)
-			(justify right)
-		)
-	)
-	(hierarchical_label "tof1_GPIO"
-		(shape input)
-		(at 63.5 128.27 180)
-		(effects
-			(font
-				(size 1.27 1.27)
-			)
-			(justify right)
-		)
-	)
-	(hierarchical_label "Bluetooth_USART3_RX"
-		(shape input)
-		(at 59.69 146.05 180)
-		(effects
-			(font
-				(size 1.27 1.27)
-			)
-			(justify right)
-		)
-	)
-	(hierarchical_label "ENC2_PH2"
-		(shape input)
-		(at 59.69 120.65 180)
-		(effects
-			(font
-				(size 1.27 1.27)
-			)
-			(justify right)
-		)
-	)
-	(hierarchical_label "PWM_Mot1_CH2"
-		(shape input)
-		(at 109.22 82.55 0)
-		(effects
-			(font
-				(size 1.27 1.27)
-			)
-			(justify left)
-		)
-	)
-	(hierarchical_label "TOF4_XSHUT"
-		(shape input)
-		(at 63.5 125.73 180)
-		(effects
-			(font
-				(size 1.27 1.27)
-			)
-			(justify right)
-		)
-	)
-	(hierarchical_label "PWM_Mot1_CH1"
-		(shape input)
-		(at 109.22 80.01 0)
-		(effects
-			(font
-				(size 1.27 1.27)
-			)
-			(justify left)
-		)
-	)
-	(hierarchical_label "PWM_Mot2_CH1"
-		(shape input)
-		(at 109.22 107.95 0)
-		(effects
-			(font
-				(size 1.27 1.27)
-			)
-			(justify left)
-		)
-	)
-	(hierarchical_label "ACC_INT2"
-		(shape input)
-		(at 59.69 148.59 180)
-		(effects
-			(font
-				(size 1.27 1.27)
-			)
-			(justify right)
-		)
-	)
-	(hierarchical_label "I2C1_SDA"
-		(shape input)
-		(at 36.83 140.97 180)
-		(effects
-			(font
-				(size 1.27 1.27)
-			)
-			(justify right)
-		)
-	)
-	(hierarchical_label "I2C1_SCL"
-		(shape input)
-		(at 31.75 138.43 180)
-		(effects
-			(font
-				(size 1.27 1.27)
-			)
-			(justify right)
-		)
-	)
-	(hierarchical_label "LIDAR_USART2_RX"
-		(shape input)
-		(at 109.22 85.09 0)
-		(effects
-			(font
-				(size 1.27 1.27)
-			)
-			(justify left)
-		)
-	)
-	(hierarchical_label "TOF2_XSHUT"
-		(shape input)
-		(at 57.15 102.87 180)
-		(effects
-			(font
-				(size 1.27 1.27)
-			)
-			(justify right)
-		)
-	)
-	(hierarchical_label "Bluetooth_USART3_TX"
-		(shape input)
-		(at 59.69 143.51 180)
-		(effects
-			(font
-				(size 1.27 1.27)
-			)
-			(justify right)
-		)
-	)
-	(hierarchical_label "M_CTR"
-		(shape input)
-		(at 114.3 100.33 0)
-		(effects
-			(font

Commit message: JJ
Connections:
- net Bluetooth_En: now reaches U1.12 (PA4)
- no-connect marks 11 -> 10
Changed lines of the file:
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@@
-	)
-	(no_connect
-		(at 100.33 90.17)
 	)
 	(no_connect
@@
 		(pts
 			(xy 176.53 123.19) (xy 176.53 127)
+		)
+		(stroke
+			(width 0)
+			(type default)
+		)
+	)
+	(wire
+		(pts
+			(xy 100.33 90.17) (xy 105.41 90.17)
 		)
 		(stroke
@@
 		(effects
 			(font
+				(size 1.27 1.27)
+			)
+			(justify left)
+		)
+	)
+	(hierarchical_label "Bluetooth_En"
+		(shape input)
+		(at 105.41 90.17 0)
+		(effects
+			(font

Commit message: s
Parts:
- added C33: 100n, Capacitor_SMD:C_0402_1005Metric, symbol Device:C_Small
- C1, C21, C5, C6, C7: value 100nF -> 100n; footprint Capacitor_SMD:C_0603_1608Metric -> Capacitor_SMD:C_0402_1005Metric
- C3, C4: value 10pF -> 10p; footprint Capacitor_SMD:C_0603_1608Metric -> Capacitor_SMD:C_0402_1005Metric
- C32: value 100nf -> 100n; footprint Capacitor_SMD:C_0201_0603Metric -> Capacitor_SMD:C_0402_1005Metric
- C8: value 10nF -> 10n
- L1: value 39nH -> 39n
- R1, R2: value 2.2K -> 2k2
- renumbered B-Res1 to SW1
Connections:
- net +3.3V: now also C33.2
- net GND: now also C33.1
Changed lines of the file:
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@@
 	(text "Bouton Chat/Souris"
 		(exclude_from_sim no)
-		(at 255.524 134.112 0)
+		(at 256.286 128.524 0)
 		(effects
 			(font
@@
 	(wire
 		(pts
+			(xy 41.91 53.34) (xy 41.91 54.61)
+		)
+		(stroke
+			(width 0)
+			(type default)
+		)
+	)
+	(wire
+		(pts
 			(xy 90.17 46.99) (xy 99.06 46.99)
 		)
@@
 	(wire
 		(pts
+			(xy 41.91 46.99) (xy 50.8 46.99)
+		)
+		(stroke
+			(width 0)
+			(type default)
+		)
+	)
+	(wire
+		(pts
 			(xy 100.33 97.79) (xy 114.3 97.79)
 		)
@@
 	(wire
 		(pts
+			(xy 41.91 48.26) (xy 41.91 46.99)
+		)
+		(stroke
+			(width 0)
+			(type default)
+		)
+	)
+	(wire
+		(pts
 			(xy 63.5 125.73) (xy 64.77 125.73)
 		)
@@
 	(wire
 		(pts
+			(xy 41.91 54.61) (xy 50.8 54.61)
+		)
+		(stroke
+			(width 0)
+			(type default)
+		)
+	)
+	(wire
+		(pts
 			(xy 276.86 149.86) (xy 276.86 151.13)
 		)
@@
 			)
 		)
-		(property "Value" "10pF"
+		(property "Value" "10p"
 			(at 40.64 85.0835 0)
 			(effects
@@
 			)
 		)
-		(property "Footprint" "Capacitor_SMD:C_0603_1608Metric"
+		(property "Footprint" "Capacitor_SMD:C_0402_1005Metric"
 			(at 38.1 83.82 0)
 			(effects
@@
 			)
 		)
-		(property "Value" "2.2K"
+		(property "Value" "2k2"
 			(at 38.608 133.604 0)
 			(effects
@@
 		(dnp no)
 		(fields_autoplaced yes)
-		(property "Reference" "B-Res1"
+		(property "Reference" "SW1"
 			(at 256.54 100.33 0)
 			(effects
@@
 			(project ""
 				(path "/21a14c86-6900-4d4b-9d91-6c59051d0f41/31be01aa-b096-4901-8c4f-f2a7c3166097"
-					(reference "B-Res1")
+					(reference "SW1")
 					(unit 1)
 				)
@@
 		(fields_autoplaced yes)
 		(property "Reference" "C4"
-			(at 35.56 104.1465 0)
+			(at 40.64 101.6062 0)
 			(effects
 				(font
 					(size 1.27 1.27)
 				)
-				(justify right)
+				(justify left)
 			)
 		)
-		(property "Value" "10pF"
-			(at 35.56 101.6065 0)
+		(property "Value" "10p"
+			(at 40.64 104.1462 0)
 			(effects
 				(font
 					(size 1.27 1.27)
 				)
-				(justify right)
+				(justify left)
 			)
 		)
-		(property "Footprint" "Capacitor_SMD:C_0603_1608Metric"
+		(property "Footprint" "Capacitor_SMD:C_0402_1005Metric"
 			(at 38.1 102.87 0)
 			(effects
@@
 			)
 		)
-		(property "Value" "100nF"
+		(property "Value" "100n"
 			(at 34.29 78.7462 0)
 			(effects
@@
 			)
 		)
-		(property "Footprint" "Capacitor_SMD:C_0603_1608Metric"
+		(property "Footprint" "Capacitor_SMD:C_0402_1005Metric"
 			(at 31.75 77.47 0)
 			(effects
@@
 			)
 		)
-		(property "Value" "10nF"
+		(property "Value" "10n"
 			(at 101.6 52.0635 0)
 			(effects
@@
 			)
 		)
-		(property "Value" "100nF"
+		(property "Value" "100n"
 			(at 69.85 52.0635 0)
 			(effects
@@
 			)
 		)
-		(property "Footprint" "Capacitor_SMD:C_0603_1608Metric"
+		(property "Footprint" "Capacitor_SMD:C_0402_1005Metric"
 			(at 67.31 50.8 0)
 			(effects
@@
 			)
 		)
-		(property "Value" "100nF"
+		(property "Value" "100n"
 			(at 77.47 52.0635 0)
 			(effects
@@
 			)
 		)
-		(property "Footprint" "Capacitor_SMD:C_0603_1608Metric"
+		(property "Footprint" "Capacitor_SMD:C_0402_1005Metric"
 			(at 74.93 50.8 0)
 			(effects
@@
 			)
 		)
-		(property "Value" "39nH"
+		(property "Value" "39n"
 			(at 86.36 44.45 90)
 			(effects
@@
 		(on_board yes)
 		(dnp no)
-		(fields_autoplaced yes)
 		(property "Reference" "ch/sou1"
-			(at 264.16 142.24 0)
+			(at 267.208 142.24 0)
 			(effects
 				(font
@@
 		)
 		(property "Value" "SW_Push"
-			(at 264.16 144.78 0)
+			(at 267.208 144.78 0)
 			(effects
 				(font
@@
 	)
 	(symbol
+		(lib_id "Device:C_Small")
+		(at 41.91 50.8 180)
+		(unit 1)
+		(exclude_from_sim no)
+		(in_bom yes)
+		(on_board yes)
+		(dnp no)
+		(fields_autoplaced yes)
+		(property "Reference" "C33"
+			(at 44.45 49.5235 0)
+			(effects
+				(font
+					(size 1.27 1.27)
+				)
+				(justify right)
+			)
+		)
+		(property "Value" "100n"
+			(at 44.45 52.0635 0)
+			(effects
+				(font
+					(size 1.27 1.27)
+				)
+				(justify right)
+			)
+		)
+		(property "Footprint" "Capacitor_SMD:C_0402_1005Metric"
+			(at 41.91 50.8 0)
+			(effects
+				(font
+					(size 1.27 1.27)
+				)
+				(hide yes)
+			)
+		)
+		(property "Datasheet" "~"
+			(at 41.91 50.8 0)
+			(effects
+				(font
+					(size 1.27 1.27)
+				)
+				(hide yes)
+			)
+		)
+		(property "Description" "Unpolarized capacitor, small symbol"
+			(at 41.91 50.8 0)
+			(effects
+				(font
+					(size 1.27 1.27)
+				)
+				(hide yes)
+			)
+		)
+		(pin "2"
+		)
+		(pin "1"
+		)
+		(instances
+			(project "Projet_Robot"
+				(path "/21a14c86-6900-4d4b-9d91-6c59051d0f41/31be01aa-b096-4901-8c4f-f2a7c3166097"
+					(reference "C33")
+					(unit 1)
+				)
+			)
+		)
+	)
+	(symbol
 		(lib_id "power:GND")
 		(at 209.55 71.12 0)
@@
 			)
 		)
-		(property "Value" "100nF"
+		(property "Value" "100n"
 			(at 57.1563 66.04 90)
 			(effects
@@
 			)
 		)
-		(property "Footprint" "Capacitor_SMD:C_0603_1608Metric"
+		(property "Footprint" "Capacitor_SMD:C_0402_1005Metric"
 			(at 57.15 69.85 0)
 			(effects
@@
 			)
 		)
-		(property "Value" "100nF"
+		(property "Value" "100n"
 			(at 62.23 52.0635 0)
 			(effects
@@
 			)
 		)
-		(property "Footprint" "Capacitor_SMD:C_0603_1608Metric"
+		(property "Footprint" "Capacitor_SMD:C_0402_1005Metric"
 			(at 59.69 50.8 0)
 			(effects
@@
 			)
 		)
-		(property "Value" "100nf"
+		(property "Value" "100n"
 			(at 246.38 157.4799 0)
 			(effects
@@
 			)
 		)
-		(property "Footprint" "Capacitor_SMD:C_0201_0603Metric"
+		(property "Footprint" "Capacitor_SMD:C_0402_1005Metric"
 			(at 243.5352 160.02 0)
 			(effects
@@
 			)
 		)
-		(property "Value" "2.2K"
+		(property "Value" "2k2"
 			(at 47.244 133.604 0)
 			(effects

Commit message: check LF
Parts:
- Y1: footprint Crystal:Crystal_SMD_0603-4Pin_6.0x3.5mm -> Crystal:Crystal_SMD_EuroQuartz_MT-4Pin_3.2x2.5mm
Changed lines of the file:
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@@
 			)
 		)
-		(property "Footprint" "Crystal:Crystal_SMD_0603-4Pin_6.0x3.5mm"
+		(property "Footprint" "Crystal:Crystal_SMD_EuroQuartz_MT-4Pin_3.2x2.5mm"
 			(at 22.86 95.25 0)
 			(effects
