File: Hardware/KiCad/capteur.kicad_sch (KiCad schematic)
At the start: 10 parts, among them IC1 ADXL343BCCZ-RL, J2 Conn_01x04, J3 Conn_01x06, J4 Conn_01x06, J5 Conn_01x05, J6 Conn_01x06, J7 Conn_01x06

Commit message: commit
Parts:
- removed J2: Conn_01x04, Connector_JST:JST_XH_B4B-XH-AM_1x04_P2.50mm_Vertical, symbol Connector_Generic:Conn_01x04
- added J1: Conn_01x05, symbol Connector_Generic:Conn_01x05
Connections:
- net +5V: now also J1.1 (Pin_1)
- net GND: now also J1.5 (Pin_5)
- net LIDAR_USART2_RX: now also J1.2 (Pin_2)
- net M_CTR: now also J1.4 (Pin_4)
- new net LIDAR_USART2_TX: J1.3 (Pin_3)

Commit message: change
Other:
- note added: "Capteurs TOF"
- note removed: "Capteur TOF 1"

Commit message: Robot
Changed lines of the file:
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@@
-		)
-	)
-	(global_label "M_CTR"
-		(shape input)
-		(at 46.99 156.21 180)
-		(fields_autoplaced yes)
-		(effects
-			(font
-				(size 1.27 1.27)
-			)
-			(justify right)
-		)
-		(property "Intersheetrefs" "${INTERSHEET_REFS}"
-			(at 38.0782 156.21 0)
-			(effects
-				(font
-					(size 1.27 1.27)
-				)
-				(justify right)
-				(hide yes)
-			)
 		)
 	)
@@
 		)
 	)
+	(hierarchical_label "M_CTR"
+		(shape input)
+		(at 46.99 156.21 180)
+		(effects
+			(font
+				(size 1.27 1.27)
+			)
+			(justify right)
+		)
+	)

Commit message: commit
Connections:
- net ACC_INT2: now reaches IC1.9 (INT2)
- removed net GPIO: IC1.8 (INT1), J3.4 (Pin_4), J4.4 (Pin_4), J6.4 (Pin_4), J7.4 (Pin_4)
- removed net XSHUT: J3.6 (Pin_6), J4.6 (Pin_6), J6.6 (Pin_6), J7.6 (Pin_6)
- new net ACC_INT1: IC1.8 (INT1)
- new net TOF1_XSHUT: J3.6 (Pin_6)
- new net TOF2_XSHUT: J4.6 (Pin_6)
- new net TOF3_XSHUT: J6.6 (Pin_6)
- new net TOF4_XSHUT: J7.6 (Pin_6)
- new net tof1_GPIO: J3.4 (Pin_4)
- new net tof2_GPIO: J4.4 (Pin_4)
- new net tof3_GPIO: J6.4 (Pin_4)
- new net tof4_GPIO: J7.4 (Pin_4)
- no-connect marks 2 -> 1
