File: Hardware/KiCad/capteur.kicad_sch (KiCad schematic)
At the start: 11 parts, among them IC1 ADXL343BCCZ-RL, J1 Conn_01x05, J3 Conn_01x06, J4 Conn_01x06, J5 Conn_01x05, J6 Conn_01x06, J7 Conn_01x06

Commit message: c
Parts:
- C26: footprint (none) -> Capacitor_SMD:C_0201_0603Metric
Changed lines of the file:
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@@
 			)
 		)
-		(property "Footprint" ""
+		(property "Footprint" "Capacitor_SMD:C_0201_0603Metric"
 			(at 92.71 152.4 0)
 			(effects

Commit message: j
Parts:
- IC1: footprint adx:ADXL343BCCZRL -> Package_LGA:LGA-14_3x5mm_P0.8mm_LayoutBorder1x6y
- J1: footprint (none) -> Battery:SOT65P280X100-8N
Changed lines of the file:
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@@
 			)
 		)
-		(property "Footprint" ""
+		(property "Footprint" "Battery:SOT65P280X100-8N"
 			(at 71.12 153.67 0)
 			(effects
@@
 			)
 		)
-		(property "Footprint" "adx:ADXL343BCCZRL"
+		(property "Footprint" "Package_LGA:LGA-14_3x5mm_P0.8mm_LayoutBorder1x6y"
 			(at 92.71 145.72 0)
 			(effects

Commit message: P
Changed lines of the file:
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@@
+	)
+	(junction
+		(at 144.78 45.72)
+		(diameter 0)
+		(color 0 0 0 0)
 	)
 	(junction
@@
 	(wire
 		(pts
-			(xy 152.4 48.26) (xy 153.67 48.26)
+			(xy 152.4 49.53) (xy 153.67 49.53)
 		)
 		(stroke
@@
 	(wire
 		(pts
-			(xy 143.51 45.72) (xy 153.67 45.72)
+			(xy 143.51 45.72) (xy 144.78 45.72)
 		)
 		(stroke
@@
 		)
 	)
+	(wire
+		(pts
+			(xy 144.78 45.72) (xy 153.67 45.72)
+		)
+		(stroke
+			(width 0)
+			(type default)
+		)
+	)
 	(bus
 		(pts
@@
 		(pts
 			(xy 43.18 85.09) (xy 43.18 76.2)
+		)
+		(stroke
+			(width 0)
+			(type default)
+		)
+	)
+	(wire
+		(pts
+			(xy 153.67 49.53) (xy 153.67 48.26)
 		)
 		(stroke
@@
 	(hierarchical_label "TOF1_XSHUT"
 		(shape input)
-		(at 152.4 48.26 180)
+		(at 152.4 49.53 180)
 		(effects
 			(font
@@
 					(unit 1)
 				)
+			)
+		)
+	)
+	(symbol
+		(lib_id "power:PWR_FLAG")
+		(at 144.78 45.72 180)
+		(unit 1)
+		(exclude_from_sim no)
+		(in_bom yes)
+		(on_board yes)
+		(dnp no)
+		(fields_autoplaced yes)
+		(property "Reference" "#FLG03"
+			(at 144.78 47.625 0)
+			(effects
+				(font
+					(size 1.27 1.27)
+				)
+				(hide yes)
+			)
+		)
+		(property "Value" "PWR_FLAG"
+			(at 144.78 50.8 0)
+			(effects
+				(font
+					(size 1.27 1.27)
+				)
+				(hide yes)
+			)
+		)
+		(property "Footprint" ""
+			(at 144.78 45.72 0)
+			(effects
+				(font
+					(size 1.27 1.27)
+				)
+				(hide yes)
+			)
+		)
+		(property "Datasheet" "~"
+			(at 144.78 45.72 0)
+			(effects
+				(font
+					(size 1.27 1.27)
+				)
+				(hide yes)
+			)
+		)
+		(property "Description" "Special symbol for telling ERC where power comes from"
+			(at 144.78 45.72 0)
+			(effects
+				(font
+					(size 1.27 1.27)
+				)
+				(hide yes)
+			)
+		)
+		(pin "1"
+		)
+		(instances
+			(project ""
+				(path "/21a14c86-6900-4d4b-9d91-6c59051d0f41/76b000bd-d8d0-4821-bef4-3e858ee71b1c"
+					(reference "#FLG03")
+					(unit 1)
+				)

Commit message: P
Parts:
- added TP5, TP6, TP7, TP8, TP9: TestPoint, symbol Connector:TestPoint
Connections:
- net ACC_INT1: now also TP8.1
- net ACC_INT2: now also TP7.1
- net I2C1_SCL: now also TP6.1
- net I2C1_SDA: now also TP5.1

Commit message: s
Parts:
- added C27, C28, C29, C30, C31: 1u, Capacitor_SMD:C_0201_0603Metric, symbol Device:C_Small
- J7: footprint Connector_JST:JST_XH_B6B-XH-AM_1x06_P2.50mm_Vertical -> Connector_JST:JST_XH_B6B-XH-A_1x06_P2.50mm_Vertical
Connections:
- net +5V: now also C27.1, C28.1, C29.1, C30.1, C31.1
- net GND: now also C27.2, C28.2, C29.2, C30.2, C31.2

Commit message: s
Parts:
- TP5, TP6, TP7, TP8, TP9: footprint (none) -> TestPoint:TestPoint_Pad_D1.5mm
Connections:
- net +3.3V: now also TP9.1
Other:
- moved on the sheet: TP9
Changed lines of the file:
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@@
 	)
 	(junction
+		(at 71.12 92.71)
+		(diameter 0)
+		(color 0 0 0 0)
+	)
+	(junction
 		(at 71.12 40.64)
 		(diameter 0)
@@
 	(wire
 		(pts
+			(xy 71.12 93.98) (xy 71.12 92.71)
+		)
+		(stroke
+			(width 0)
+			(type default)
+		)
+	)
+	(wire
+		(pts
 			(xy 71.12 40.64) (xy 71.12 43.18)
 		)
@@
 	(wire
 		(pts
+			(xy 71.12 92.71) (xy 71.12 91.44)
+		)
+		(stroke
+			(width 0)
+			(type default)
+		)
+	)
+	(wire
+		(pts
 			(xy 96.52 63.5) (xy 105.41 63.5)
 		)
@@
 			)
 		)
-		(property "Footprint" ""
+		(property "Footprint" "TestPoint:TestPoint_Pad_D1.5mm"
 			(at 104.14 73.66 0)
 			(effects
@@
 			)
 		)
-		(property "Footprint" ""
+		(property "Footprint" "TestPoint:TestPoint_Pad_D1.5mm"
 			(at 110.49 63.5 0)
 			(effects
@@
 	(symbol
 		(lib_id "Connector:TestPoint")
-		(at 71.12 88.9 90)
+		(at 71.12 92.71 90)
 		(unit 1)
 		(exclude_from_sim no)
@@
 		(fields_autoplaced yes)
 		(property "Reference" "TP9"
-			(at 67.818 83.82 90)
+			(at 67.818 87.63 90)
 			(effects
 				(font
@@
 		)
 		(property "Value" "TestPoint"
-			(at 67.818 86.36 90)
+			(at 67.818 90.17 90)
 			(effects
 				(font
@@
 			)
 		)
-		(property "Footprint" ""
-			(at 71.12 83.82 0)
+		(property "Footprint" "TestPoint:TestPoint_Pad_D1.5mm"
+			(at 71.12 87.63 0)
 			(effects
 				(font
@@
 		)
 		(property "Datasheet" "~"
-			(at 71.12 83.82 0)
+			(at 71.12 87.63 0)
 			(effects
 				(font
@@
 		)
 		(property "Description" "test point"
-			(at 71.12 88.9 0)
+			(at 71.12 92.71 0)
 			(effects
 				(font
@@
 			)
 		)
-		(property "Footprint" ""
+		(property "Footprint" "TestPoint:TestPoint_Pad_D1.5mm"
 			(at 71.12 35.56 0)
 			(effects
@@
 	(symbol
 		(lib_id "power:+3.3V")
-		(at 71.12 91.44 180)
+		(at 71.12 93.98 180)
 		(unit 1)
 		(exclude_from_sim no)
@@
 		(fields_autoplaced yes)
 		(property "Reference" "#PWR0130"
-			(at 71.12 87.63 0)
+			(at 71.12 90.17 0)
 			(effects
 				(font
@@
 		)
 		(property "Value" "+3.3V"
-			(at 71.12 96.52 0)
+			(at 71.12 99.06 0)
 			(effects
 				(font
@@
 		)
 		(property "Footprint" ""
-			(at 71.12 91.44 0)
+			(at 71.12 93.98 0)
 			(effects
 				(font
@@
 		)
 		(property "Datasheet" ""
-			(at 71.12 91.44 0)
+			(at 71.12 93.98 0)
 			(effects
 				(font
@@
 		)
 		(property "Description" "Power symbol creates a global label with name \"+3.3V\""
-			(at 71.12 91.44 0)
+			(at 71.12 93.98 0)
 			(effects
 				(font
@@
 			)
 		)
-		(property "Footprint" ""
+		(property "Footprint" "TestPoint:TestPoint_Pad_D1.5mm"
 			(at 93.98 76.2 0)
 			(effects

Commit message: hhhh
Parts:
- J3, J4, J6: footprint Connector_JST:JST_XH_B6B-XH-AM_1x06_P2.50mm_Vertical -> Connector_JST:JST_XH_B6B-XH-A_1x06_P2.50mm_Vertical
Changed lines of the file:
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@@
 			)
 		)
-		(property "Footprint" "Connector_JST:JST_XH_B6B-XH-AM_1x06_P2.50mm_Vertical"
+		(property "Footprint" "Connector_JST:JST_XH_B6B-XH-A_1x06_P2.50mm_Vertical"
 			(at 195.58 40.64 0)
 			(effects
@@
 			)
 		)
-		(property "Footprint" "Connector_JST:JST_XH_B6B-XH-AM_1x06_P2.50mm_Vertical"
+		(property "Footprint" "Connector_JST:JST_XH_B6B-XH-A_1x06_P2.50mm_Vertical"
 			(at 158.75 40.64 0)
 			(effects
@@
 			)
 		)
-		(property "Footprint" "Connector_JST:JST_XH_B6B-XH-AM_1x06_P2.50mm_Vertical"
+		(property "Footprint" "Connector_JST:JST_XH_B6B-XH-A_1x06_P2.50mm_Vertical"
 			(at 236.22 40.64 0)
 			(effects

Commit message: s
s
Parts:
- removed J5: Conn_01x05, Connector_JST:JST_XH_B6B-XH-AM_1x06_P2.50mm_Vertical, symbol Connector_Generic:Conn_01x05
- added J9: Conn_01x06, Connector_PinSocket_2.54mm:PinSocket_1x06_P2.54mm_Vertical, symbol Connector_Generic:Conn_01x06
- J1: footprint Battery:SOT65P280X100-8N -> Connector_JST:JST_XH_B5B-XH-A_1x05_P2.50mm_Vertical
Connections:
- net +5V: now also J9.2 (Pin_2)
- net Bluetooth_USART3_RX: now also J9.5 (Pin_5)
- net Bluetooth_USART3_TX: now also J9.4 (Pin_4)
- net GND: now also J9.3 (Pin_3)
- new net Bluetooth_En: J9.1 (Pin_1)
