File: Hardware/KiCad/capteur.kicad_sch (KiCad schematic)
At the start: 21 parts, among them IC1 ADXL343BCCZ-RL, J1 Conn_01x05, J3 Conn_01x06, J4 Conn_01x06, J6 Conn_01x06, J7 Conn_01x06, J9 Conn_01x06

Commit message: w
Parts:
- renumbered J9 to Bluetooth1, J1 to Lidar1, J3 to TOF1, J4 to TOF2, J6 to TOF3, J7 to TOF4
Changed lines of the file:
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@@
 		(dnp no)
 		(fields_autoplaced yes)
-		(property "Reference" "J7"
+		(property "Reference" "TOF4"
 			(at 273.05 40.6399 0)
 			(effects
@@
 			(project "Projet_Robot"
 				(path "/21a14c86-6900-4d4b-9d91-6c59051d0f41/76b000bd-d8d0-4821-bef4-3e858ee71b1c"
-					(reference "J7")
+					(reference "TOF4")
 					(unit 1)
 				)
@@
 		(dnp no)
 		(fields_autoplaced yes)
-		(property "Reference" "J4"
+		(property "Reference" "TOF2"
 			(at 198.12 40.6399 0)
 			(effects
@@
 			(project "Projet_Robot"
 				(path "/21a14c86-6900-4d4b-9d91-6c59051d0f41/76b000bd-d8d0-4821-bef4-3e858ee71b1c"
-					(reference "J4")
+					(reference "TOF2")
 					(unit 1)
 				)
@@
 		(dnp no)
 		(fields_autoplaced yes)
-		(property "Reference" "J3"
+		(property "Reference" "TOF1"
 			(at 161.29 40.6399 0)
 			(effects
@@
 			(project ""
 				(path "/21a14c86-6900-4d4b-9d91-6c59051d0f41/76b000bd-d8d0-4821-bef4-3e858ee71b1c"
-					(reference "J3")
+					(reference "TOF1")
 					(unit 1)
 				)
@@
 		(dnp no)
 		(fields_autoplaced yes)
-		(property "Reference" "J9"
+		(property "Reference" "Bluetooth1"
 			(at 208.28 92.7099 0)
 			(effects
@@
 			(project "Projet_Robot"
 				(path "/21a14c86-6900-4d4b-9d91-6c59051d0f41/76b000bd-d8d0-4821-bef4-3e858ee71b1c"
-					(reference "J9")
+					(reference "Bluetooth1")
 					(unit 1)
 				)
@@
 		(dnp no)
 		(fields_autoplaced yes)
-		(property "Reference" "J6"
+		(property "Reference" "TOF3"
 			(at 238.76 40.6399 0)
 			(effects
@@
 			(project "Projet_Robot"
 				(path "/21a14c86-6900-4d4b-9d91-6c59051d0f41/76b000bd-d8d0-4821-bef4-3e858ee71b1c"
-					(reference "J6")
+					(reference "TOF3")
 					(unit 1)
 				)
@@
 		(dnp no)
 		(fields_autoplaced yes)
-		(property "Reference" "J1"
+		(property "Reference" "Lidar1"
 			(at 73.66 152.3999 0)
 			(effects
@@
 			(project ""
 				(path "/21a14c86-6900-4d4b-9d91-6c59051d0f41/76b000bd-d8d0-4821-bef4-3e858ee71b1c"
-					(reference "J1")
-					(unit 1)
-				)
+					(reference "Lidar1")
+					(unit 1)
+				)

Commit message: s
Parts:
- removed TP5, TP9: TestPoint, TestPoint:TestPoint_Pad_D1.5mm, symbol Connector:TestPoint
Changed lines of the file:
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@@
-	)
-	(junction
-		(at 71.12 92.71)
-		(diameter 0)
-		(color 0 0 0 0)
 	)
 	(junction
@@
 	)
 	(junction
-		(at 105.41 63.5)
-		(diameter 0)
-		(color 0 0 0 0)
-	)
-	(junction
 		(at 30.48 76.2)
 		(diameter 0)
@@
 	(wire
 		(pts
-			(xy 71.12 93.98) (xy 71.12 92.71)
+			(xy 71.12 91.44) (xy 71.12 93.98)
 		)
 		(stroke
@@
 	(wire
 		(pts
-			(xy 71.12 92.71) (xy 71.12 91.44)
-		)
-		(stroke
-			(width 0)
-			(type default)
-		)
-	)
-	(wire
-		(pts
-			(xy 96.52 63.5) (xy 105.41 63.5)
+			(xy 96.52 63.5) (xy 110.49 63.5)
 		)
 		(stroke
@@
 		(pts
 			(xy 228.6 48.26) (xy 231.14 48.26)
-		)
-		(stroke
-			(width 0)
-			(type default)
-		)
-	)
-	(wire
-		(pts
-			(xy 105.41 63.5) (xy 110.49 63.5)
 		)
 		(stroke
@@
 					(unit 1)
 				)
-			)
-		)
-	)
-	(symbol
-		(lib_id "Connector:TestPoint")
-		(at 105.41 63.5 0)
-		(unit 1)
-		(exclude_from_sim no)
-		(in_bom yes)
-		(on_board yes)
-		(dnp no)
-		(fields_autoplaced yes)
-		(property "Reference" "TP5"
-			(at 107.95 58.9279 0)
-			(effects
-				(font
-					(size 1.27 1.27)
-				)
-				(justify left)
-			)
-		)
-		(property "Value" "TestPoint"
-			(at 107.95 61.4679 0)
-			(effects
-				(font
-					(size 1.27 1.27)
-				)
-				(justify left)
-			)
-		)
-		(property "Footprint" "TestPoint:TestPoint_Pad_D1.5mm"
-			(at 110.49 63.5 0)
-			(effects
-				(font
-					(size 1.27 1.27)
-				)
-				(hide yes)
-			)
-		)
-		(property "Datasheet" "~"
-			(at 110.49 63.5 0)
-			(effects
-				(font
-					(size 1.27 1.27)
-				)
-				(hide yes)
-			)
-		)
-		(property "Description" "test point"
-			(at 105.41 63.5 0)
-			(effects
-				(font
-					(size 1.27 1.27)
-				)
-				(hide yes)
-			)
-		)
-		(pin "1"
-		)
-		(instances
-			(project ""
-				(path "/21a14c86-6900-4d4b-9d91-6c59051d0f41/76b000bd-d8d0-4821-bef4-3e858ee71b1c"
-					(reference "TP5")
-					(unit 1)
-				)
-			)
-		)
-	)
-	(symbol
-		(lib_id "Connector:TestPoint")
-		(at 71.12 92.71 90)
-		(unit 1)
-		(exclude_from_sim no)
-		(in_bom yes)
-		(on_board yes)
-		(dnp no)
-		(fields_autoplaced yes)
-		(property "Reference" "TP9"
-			(at 67.818 87.63 90)
-			(effects
-				(font
-					(size 1.27 1.27)
-				)
-			)
-		)
-		(property "Value" "TestPoint"
-			(at 67.818 90.17 90)
-			(effects
-				(font
-					(size 1.27 1.27)
-				)
-			)
-		)
-		(property "Footprint" "TestPoint:TestPoint_Pad_D1.5mm"
-			(at 71.12 87.63 0)
-			(effects
-				(font
-					(size 1.27 1.27)
-				)
-				(hide yes)
-			)
-		)
-		(property "Datasheet" "~"
-			(at 71.12 87.63 0)
-			(effects
-				(font
-					(size 1.27 1.27)
-				)
-				(hide yes)
-			)
-		)
-		(property "Description" "test point"
-			(at 71.12 92.71 0)
-			(effects
-				(font
-					(size 1.27 1.27)
-				)
-				(hide yes)
-			)
-		)
-		(pin "1"
-		)
-		(instances
-			(project ""
-				(path "/21a14c86-6900-4d4b-9d91-6c59051d0f41/76b000bd-d8d0-4821-bef4-3e858ee71b1c"
-					(reference "TP9")
-					(unit 1)
-				)

Commit message: s
Parts:
- C11, C9: value 0.1u -> 100n; footprint Capacitor_SMD:C_0603_1608Metric -> Capacitor_SMD:C_0402_1005Metric
- C26, C27, C28, C29, C30, C31: footprint Capacitor_SMD:C_0201_0603Metric -> Capacitor_SMD:C_0603_1608Metric
- TOF1, TOF2, TOF3, TOF4: footprint Connector_JST:JST_XH_B6B-XH-A_1x06_P2.50mm_Vertical -> Connector_PinSocket_2.54mm:PinSocket_1x06_P2.54mm_Vertical
Connections:
- net Bluetooth_USART3_RX: now also Bluetooth1.4 (Pin_4); no longer Bluetooth1.5 (Pin_5)
- net Bluetooth_USART3_TX: now also Bluetooth1.5 (Pin_5); no longer Bluetooth1.4 (Pin_4)
Changed lines of the file:
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@@
 		)
 	)
+	(hierarchical_label "Bluetooth_USART3_TX"
+		(shape input)
+		(at 200.66 97.79 180)
+		(effects
+			(font
+				(size 1.27 1.27)
+			)
+			(justify right)
+		)
+	)
 	(hierarchical_label "tof2_GPIO"
 		(shape input)
@@
 	(hierarchical_label "Bluetooth_USART3_RX"
 		(shape input)
-		(at 200.66 97.79 180)
+		(at 200.66 95.25 180)
 		(effects
 			(font
@@
 		)
 	)
-	(hierarchical_label "Bluetooth_USART3_TX"
-		(shape input)
-		(at 200.66 95.25 180)
-		(effects
-			(font
-				(size 1.27 1.27)
-			)
-			(justify right)
-		)
-	)
 	(hierarchical_label "I2C1_SCL"
 		(shape input)
@@
 			)
 		)
-		(property "Footprint" "Connector_JST:JST_XH_B6B-XH-A_1x06_P2.50mm_Vertical"
+		(property "Footprint" "Connector_PinSocket_2.54mm:PinSocket_1x06_P2.54mm_Vertical"
 			(at 270.51 40.64 0)
 			(effects
@@
 			)
 		)
-		(property "Footprint" "Connector_JST:JST_XH_B6B-XH-A_1x06_P2.50mm_Vertical"
+		(property "Footprint" "Connector_PinSocket_2.54mm:PinSocket_1x06_P2.54mm_Vertical"
 			(at 195.58 40.64 0)
 			(effects
@@
 			)
 		)
-		(property "Footprint" "Capacitor_SMD:C_0201_0603Metric"
+		(property "Footprint" "Capacitor_SMD:C_0603_1608Metric"
 			(at 92.71 152.4 0)
 			(effects
@@
 			)
 		)
-		(property "Footprint" "Connector_JST:JST_XH_B6B-XH-A_1x06_P2.50mm_Vertical"
+		(property "Footprint" "Connector_PinSocket_2.54mm:PinSocket_1x06_P2.54mm_Vertical"
 			(at 158.75 40.64 0)
 			(effects
@@
 			)
 		)
-		(property "Footprint" "Capacitor_SMD:C_0201_0603Metric"
+		(property "Footprint" "Capacitor_SMD:C_0603_1608Metric"
 			(at 242.57 33.02 0)
 			(effects
@@
 			)
 		)
-		(property "Value" "0.1u"
+		(property "Value" "100n"
 			(at 36.83 58.42 90)
 			(effects
@@
 			)
 		)
-		(property "Footprint" "Capacitor_SMD:C_0603_1608Metric"
+		(property "Footprint" "Capacitor_SMD:C_0402_1005Metric"
 			(at 40.64 62.5348 0)
 			(effects
@@
 			)
 		)
-		(property "Footprint" "Capacitor_SMD:C_0201_0603Metric"
+		(property "Footprint" "Capacitor_SMD:C_0603_1608Metric"
 			(at 166.37 33.02 0)
 			(effects
@@
 			)
 		)
-		(property "Footprint" "Connector_JST:JST_XH_B6B-XH-A_1x06_P2.50mm_Vertical"
+		(property "Footprint" "Connector_PinSocket_2.54mm:PinSocket_1x06_P2.54mm_Vertical"
 			(at 236.22 40.64 0)
 			(effects
@@
 			)
 		)
-		(property "Footprint" "Capacitor_SMD:C_0201_0603Metric"
+		(property "Footprint" "Capacitor_SMD:C_0603_1608Metric"
 			(at 204.47 33.02 0)
 			(effects
@@
 			)
 		)
-		(property "Footprint" "Capacitor_SMD:C_0201_0603Metric"
+		(property "Footprint" "Capacitor_SMD:C_0603_1608Metric"
 			(at 234.95 91.44 0)
 			(effects
@@
 			)
 		)
-		(property "Footprint" "Capacitor_SMD:C_0201_0603Metric"
+		(property "Footprint" "Capacitor_SMD:C_0603_1608Metric"
 			(at 276.86 33.02 0)
 			(effects
@@
 			)
 		)
-		(property "Value" "0.1u"
+		(property "Value" "100n"
 			(at 36.83 91.186 90)
 			(effects
@@
 			)
 		)
-		(property "Footprint" "Capacitor_SMD:C_0603_1608Metric"
+		(property "Footprint" "Capacitor_SMD:C_0402_1005Metric"
 			(at 40.64 84.1248 0)
 			(effects

Commit message: R
Changed lines of the file:
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@@
 		(lib_id "Device:C_Small")
 		(at 92.71 152.4 0)
+		(mirror y)
 		(unit 1)
 		(exclude_from_sim no)
@@
 		(on_board yes)
 		(dnp no)
-		(fields_autoplaced yes)
 		(property "Reference" "C26"
-			(at 95.25 151.1362 0)
+			(at 90.17 151.1362 0)
 			(effects
 				(font
@@
 		)
 		(property "Value" "1u"
-			(at 95.25 153.6762 0)
+			(at 90.17 153.6762 0)
 			(effects
 				(font

Commit message: check LF
Connections:
- net +3.3V: now also C10.2, C11.2, C27.1, C28.1, C29.1, C30.1, C9.2, IC1.1 (VDD_I/O), IC1.3 (RESERVED_1), IC1.6 (VS), TOF1.1 (Pin_1), TOF2.1 (Pin_1), TOF3.1 (Pin_1), TOF4.1 (Pin_1); no longer C10.1, C11.1, C9.1
- net +5V: no longer C27.1, C28.1, C29.1, C30.1, TOF1.1 (Pin_1), TOF2.1 (Pin_1), TOF3.1 (Pin_1), TOF4.1 (Pin_1)
- net GND: now also C10.1, C11.1, C9.1
Other:
- moved on the sheet: C10, C11, C9
