File: Hardware/KiCad/Projet_Robot.kicad_sch (KiCad schematic)
At the start: 0 parts

Commit message: commit
Other:
- sheet Capteurs ports: added Bluetooth_USART3_RX, Bluetooth_USART3_TX, LIDAR_USART2_RX, LIDAR_USART2_TX; removed none
- sheet µcontrolleur ports: added Bluetooth_USART3_RX, Bluetooth_USART3_TX, LIDAR_USART2_RX, LIDAR_USART2_TX; removed none
Changed lines of the file:
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@@
 	(generator_version "9.0")
 	(paper "A4")
+	(wire
+		(pts
+			(xy 100.33 46.99) (xy 118.11 46.99)
+		)
+		(stroke
+			(width 0)
+			(type default)
+		)
+	)
+	(wire
+		(pts
+			(xy 100.33 34.29) (xy 118.11 34.29)
+		)
+		(stroke
+			(width 0)
+			(type default)
+		)
+	)
+	(wire
+		(pts
+			(xy 100.33 43.18) (xy 118.11 43.18)
+		)
+		(stroke
+			(width 0)
+			(type default)
+		)
+	)
+	(wire
+		(pts
+			(xy 100.33 30.48) (xy 118.11 30.48)
+		)
+		(stroke
+			(width 0)
+			(type default)
+		)
+	)
 	(sheet
 		(at 21.59 20.32)
@@
 				)
 				(justify left top)
+			)
+		)
+		(pin "LIDAR_USART2_RX" input
+			(at 100.33 30.48 0)
+			(effects
+				(font
+					(size 1.27 1.27)
+				)
+				(justify right)
+			)
+		)
+		(pin "LIDAR_USART2_TX" input
+			(at 100.33 34.29 0)
+			(effects
+				(font
+					(size 1.27 1.27)
+				)
+				(justify right)
+			)
+		)
+		(pin "Bluetooth_USART3_RX" input
+			(at 100.33 43.18 0)
+			(effects
+				(font
+					(size 1.27 1.27)
+				)
+				(justify right)
+			)
+		)
+		(pin "Bluetooth_USART3_TX" input
+			(at 100.33 46.99 0)
+			(effects
+				(font
+					(size 1.27 1.27)
+				)
+				(justify right)
 			)
 		)
@@
 			)
 		)
+		(pin "LIDAR_USART2_RX" input
+			(at 118.11 30.48 180)
+			(effects
+				(font
+					(size 1.27 1.27)
+				)
+				(justify left)
+			)
+		)
+		(pin "LIDAR_USART2_TX" input
+			(at 118.11 34.29 180)
+			(effects
+				(font
+					(size 1.27 1.27)
+				)
+				(justify left)
+			)
+		)
+		(pin "Bluetooth_USART3_RX" input
+			(at 118.11 43.18 180)
+			(effects
+				(font
+					(size 1.27 1.27)
+				)
+				(justify left)
+			)
+		)
+		(pin "Bluetooth_USART3_TX" input
+			(at 118.11 46.99 180)
+			(effects
+				(font
+					(size 1.27 1.27)
+				)
+				(justify left)
+			)
+		)

Commit message: change
Other:
- sheet Capteurs ports: added I2C1_SCL, I2C1_SDA; removed none
- sheet µcontrolleur ports: added I2C1_SCL, I2C1_SDA; removed none
Changed lines of the file:
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@@
+	(wire
+		(pts
+			(xy 100.33 57.15) (xy 118.11 57.15)
+		)
+		(stroke
+			(width 0)
+			(type default)
+		)
+	)
 	(wire
 		(pts
@@
 		(pts
 			(xy 100.33 43.18) (xy 118.11 43.18)
+		)
+		(stroke
+			(width 0)
+			(type default)
+		)
+	)
+	(wire
+		(pts
+			(xy 100.33 54.61) (xy 118.11 54.61)
 		)
 		(stroke
@@
 			)
 		)
+		(pin "I2C1_SCL" input
+			(at 100.33 54.61 0)
+			(effects
+				(font
+					(size 1.27 1.27)
+				)
+				(justify right)
+			)
+		)
+		(pin "I2C1_SDA" input
+			(at 100.33 57.15 0)
+			(effects
+				(font
+					(size 1.27 1.27)
+				)
+				(justify right)
+			)
+		)
 		(instances
 			(project "Projet_Robot"
@@
 			(effects
 				(font
+					(size 1.27 1.27)
+				)
+				(justify left)
+			)
+		)
+		(pin "I2C1_SCL" input
+			(at 118.11 54.61 180)
+			(effects
+				(font
+					(size 1.27 1.27)
+				)
+				(justify left)
+			)
+		)
+		(pin "I2C1_SDA" input
+			(at 118.11 57.15 180)
+			(effects
+				(font

Commit message: change
Other:
- removed sheet Moteur
- added sheet Moteur1 (moteur1.kicad_sch)
- added sheet Moteur2 (moteur2.kicad_sch)
- sheet µcontrolleur ports: added ENC1_PH1, ENC1_PH2, ENC2_PH1, ENC2_PH2, PWM_Mot1_CH1, PWM_Mot1_CH2, PWM_Mot2_CH1, PWM_Mot2_CH2; removed none

Commit message: Robot
Other:
- sheet Capteurs ports: added M_CTR; removed none
- sheet µcontrolleur ports: added M_CTR; removed none

Commit message: commit
Other:
- sheet Capteurs ports: added ACC_INT1, ACC_INT2, TOF1_XSHUT, TOF2_XSHUT, TOF3_XSHUT, TOF4_XSHUT, tof1_GPIO, tof2_GPIO, tof3_GPIO, tof4_GPIO; removed none
- sheet µcontrolleur ports: added ACC_INT1, ACC_INT2, TOF1_XSHUT, TOF2_XSHUT, TOF3_XSHUT, TOF4_XSHUT, tof1_GPIO, tof2_GPIO, tof3_GPIO, tof4_GPIO; removed none

Commit message: review pcb
Other:
- sheet Moteur2: file moteur2.kicad_sch -> moteur1.kicad_sch
- sheet Moteur2 ports: added ENC1_PH1, ENC1_PH2, PWM_Mot1_CH1, PWM_Mot1_CH2; removed ENC2_PH1, ENC2_PH2, PWM_Mot2_CH1, PWM_Mot2_CH2
Changed lines of the file:
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@@
+	(wire
+		(pts
+			(xy 73.66 96.52) (xy 87.63 96.52)
+		)
+		(stroke
+			(width 0)
+			(type default)
+		)
+	)
 	(wire
 		(pts
@@
 	(wire
 		(pts
-			(xy 74.93 113.03) (xy 87.63 113.03)
-		)
-		(stroke
-			(width 0)
-			(type default)
-		)
-	)
-	(wire
-		(pts
 			(xy 233.68 121.92) (xy 193.04 121.92)
 		)
@@
 	(wire
 		(pts
+			(xy 73.66 118.11) (xy 87.63 118.11)
+		)
+		(stroke
+			(width 0)
+			(type default)
+		)
+	)
+	(wire
+		(pts
+			(xy 73.66 86.36) (xy 87.63 86.36)
+		)
+		(stroke
+			(width 0)
+			(type default)
+		)
+	)
+	(wire
+		(pts
 			(xy 233.68 106.68) (xy 185.42 106.68)
 		)
@@
 	(wire
 		(pts
+			(xy 73.66 88.9) (xy 87.63 88.9)
+		)
+		(stroke
+			(width 0)
+			(type default)
+		)
+	)
+	(wire
+		(pts
 			(xy 165.1 80.01) (xy 173.99 80.01)
 		)
@@
 	(wire
 		(pts
-			(xy 165.1 153.67) (xy 238.76 153.67)
-		)
-		(stroke
-			(width 0)
-			(type default)
-		)
-	)
-	(wire
-		(pts
 			(xy 165.1 116.84) (xy 189.23 116.84)
 		)
@@
 	(wire
 		(pts
-			(xy 181.61 157.48) (xy 165.1 157.48)
-		)
-		(stroke
-			(width 0)
-			(type default)
-		)
-	)
-	(wire
-		(pts
 			(xy 184.15 101.6) (xy 184.15 104.14)
 		)
@@
 	(wire
 		(pts
-			(xy 74.93 105.41) (xy 87.63 105.41)
+			(xy 73.66 115.57) (xy 87.63 115.57)
 		)
 		(stroke
@@
 	(wire
 		(pts
-			(xy 165.1 163.83) (xy 238.76 163.83)
-		)
-		(stroke
-			(width 0)
-			(type default)
-		)
-	)
-	(wire
-		(pts
 			(xy 185.42 106.68) (xy 185.42 110.49)
 		)
@@
 	(wire
 		(pts
-			(xy 74.93 110.49) (xy 87.63 110.49)
+			(xy 73.66 123.19) (xy 87.63 123.19)
 		)
 		(stroke
@@
 	(wire
 		(pts
-			(xy 181.61 156.21) (xy 238.76 156.21)
-		)
-		(stroke
-			(width 0)
-			(type default)
-		)
-	)
-	(wire
-		(pts
 			(xy 191.77 119.38) (xy 191.77 123.19)
 		)
@@
 	(wire
 		(pts
+			(xy 73.66 125.73) (xy 87.63 125.73)
+		)
+		(stroke
+			(width 0)
+			(type default)
+		)
+	)
+	(wire
+		(pts
 			(xy 165.1 71.12) (xy 204.47 71.12)
 		)
@@
 	(wire
 		(pts
-			(xy 74.93 102.87) (xy 87.63 102.87)
+			(xy 73.66 93.98) (xy 87.63 93.98)
 		)
 		(stroke
@@
 	(wire
 		(pts
-			(xy 181.61 156.21) (xy 181.61 157.48)
-		)
-		(stroke
-			(width 0)
-			(type default)
-		)
-	)
-	(wire
-		(pts
 			(xy 190.5 115.57) (xy 190.5 119.38)
 		)
@@
 		)
 	)
-	(wire
-		(pts
-			(xy 165.1 161.29) (xy 238.76 161.29)
-		)
-		(stroke
-			(width 0)
-			(type default)
-		)
-	)
 	(sheet
-		(at 238.76 149.86)
+		(at 39.37 82.55)
 		(size 34.29 17.78)
 		(exclude_from_sim no)
@@
 		)
 		(property "Sheetname" "Moteur1"
-			(at 238.76 147.8784 0)
+			(at 39.37 80.5684 0)
 			(effects
 				(font
@@
 		)
 		(property "Sheetfile" "moteur1.kicad_sch"
-			(at 238.76 168.2246 0)
+			(at 39.37 100.9146 0)
 			(effects
 				(font
@@
 		)
 		(pin "ENC1_PH1" input
-			(at 238.76 161.29 180)
-			(effects
-				(font
-					(size 1.27 1.27)
-				)
-				(justify left)
+			(at 73.66 86.36 0)
+			(effects
+				(font
+					(size 1.27 1.27)
+				)
+				(justify right)
 			)
 		)
 		(pin "ENC1_PH2" input
-			(at 238.76 163.83 180)
-			(effects
-				(font
-					(size 1.27 1.27)
-				)
-				(justify left)
+			(at 73.66 88.9 0)
+			(effects
+				(font
+					(size 1.27 1.27)
+				)
+				(justify right)
 			)
 		)
 		(pin "PWM_Mot1_CH1" input
-			(at 238.76 153.67 180)
-			(effects
-				(font
-					(size 1.27 1.27)
-				)
-				(justify left)
+			(at 73.66 93.98 0)
+			(effects
+				(font
+					(size 1.27 1.27)
+				)
+				(justify right)
 			)
 		)
 		(pin "PWM_Mot1_CH2" input
-			(at 238.76 156.21 180)
-			(effects
-				(font
-					(size 1.27 1.27)
-				)
-				(justify left)
+			(at 73.66 96.52 0)
+			(effects
+				(font
+					(size 1.27 1.27)
+				)
+				(justify right)
 			)
 		)
@@
 		)
 		(pin "ENC1_PH1" input
-			(at 165.1 161.29 0)
-			(effects
-				(font
-					(size 1.27 1.27)
-				)
-				(justify right)
+			(at 87.63 86.36 180)
+			(effects
+				(font
+					(size 1.27 1.27)
+				)
+				(justify left)
 			)
 		)
 		(pin "ENC1_PH2" input
-			(at 165.1 163.83 0)
-			(effects
-				(font
-					(size 1.27 1.27)
-				)
-				(justify right)
+			(at 87.63 88.9 180)
+			(effects
+				(font
+					(size 1.27 1.27)
+				)
+				(justify left)
 			)
 		)
 		(pin "ENC2_PH1" input
-			(at 87.63 110.49 180)
+			(at 87.63 115.57 180)
 			(effects
 				(font
@@
 		)
 		(pin "ENC2_PH2" input
-			(at 87.63 113.03 180)
+			(at 87.63 118.11 180)
 			(effects
 				(font
@@
 		)
 		(pin "PWM_Mot1_CH1" input
-			(at 165.1 153.67 0)
-			(effects
-				(font
-					(size 1.27 1.27)
-				)
-				(justify right)
+			(at 87.63 93.98 180)
+			(effects
+				(font
+					(size 1.27 1.27)
+				)
+				(justify left)
 			)
 		)
 		(pin "PWM_Mot1_CH2" input
-			(at 165.1 157.48 0)
-			(effects
-				(font
-					(size 1.27 1.27)
-				)
-				(justify right)
+			(at 87.63 96.52 180)
+			(effects
+				(font
+					(size 1.27 1.27)
+				)
+				(justify left)
 			)
 		)
 		(pin "PWM_Mot2_CH1" input
-			(at 87.63 102.87 180)
+			(at 87.63 123.19 180)
 			(effects
 				(font
@@
 		)
 		(pin "PWM_Mot2_CH2" input
-			(at 87.63 105.41 180)
+			(at 87.63 125.73 180)
 			(effects
 				(font
@@
 	)
 	(sheet
-		(at 40.64 96.52)
-		(size 34.29 20.32)
+		(at 39.37 111.76)
+		(size 34.29 17.78)
 		(exclude_from_sim no)
 		(in_bom yes)
@@
 		)
 		(property "Sheetname" "Moteur2"
-			(at 40.64 94.5384 0)
+			(at 39.37 109.7784 0)
 			(effects
 				(font
@@
 			)
 		)
-		(property "Sheetfile" "moteur2.kicad_sch"
-			(at 40.64 117.4246 0)
+		(property "Sheetfile" "moteur1.kicad_sch"
+			(at 39.37 130.1246 0)
 			(effects
 				(font
@@
 			)
 		)
-		(pin "ENC2_PH1" input
-			(at 74.93 110.49 0)
-			(effects
-				(font
-					(size 1.27 1.27)
-				)
-				(justify right)
-			)
-		)
-		(pin "ENC2_PH2" input
-			(at 74.93 113.03 0)
-			(effects
-				(font
-					(size 1.27 1.27)
-				)
-				(justify right)
-			)
-		)
-		(pin "PWM_Mot2_CH1" input
-			(at 74.93 102.87 0)
-			(effects
-				(font
-					(size 1.27 1.27)
-				)
-				(justify right)
-			)
-		)
-		(pin "PWM_Mot2_CH2" input
-			(at 74.93 105.41 0)
+		(pin "ENC1_PH1" input
+			(at 73.66 115.57 0)
+			(effects
+				(font
+					(size 1.27 1.27)
+				)
+				(justify right)
+			)
+		)
+		(pin "ENC1_PH2" input
+			(at 73.66 118.11 0)
+			(effects
+				(font
+					(size 1.27 1.27)
+				)
+				(justify right)
+			)
+		)
+		(pin "PWM_Mot1_CH1" input
+			(at 73.66 123.19 0)
+			(effects
+				(font
+					(size 1.27 1.27)
+				)
+				(justify right)
+			)
+		)
+		(pin "PWM_Mot1_CH2" input
+			(at 73.66 125.73 0)
 			(effects
 				(font
@@
 			(project "Projet_Robot"
 				(path "/21a14c86-6900-4d4b-9d91-6c59051d0f41"
-					(page "6")
-				)
-			)
+					(page "5")
+				)
+			)

Commit message: update
Other:
- sheet Capteurs ports: added none; removed LIDAR_USART2_TX
- sheet µcontrolleur ports: added none; removed LIDAR_USART2_TX
Changed lines of the file:
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@@
+	(wire
+		(pts
+			(xy 165.1 68.58) (xy 220.98 68.58)
+		)
+		(stroke
+			(width 0)
+			(type default)
+		)
+	)
+	(wire
+		(pts
+			(xy 73.66 93.98) (xy 87.63 93.98)
+		)
+		(stroke
+			(width 0)
+			(type default)
+		)
+	)
+	(wire
+		(pts
+			(xy 165.1 82.55) (xy 220.98 82.55)
+		)
+		(stroke
+			(width 0)
+			(type default)
+		)
+	)
 	(wire
 		(pts
 			(xy 165.1 71.12) (xy 220.98 71.12)
-		)
-		(stroke
-			(width 0)
-			(type default)
-		)
-	)
-	(wire
-		(pts
-			(xy 165.1 68.58) (xy 220.98 68.58)
-		)
-		(stroke
-			(width 0)
-			(type default)
-		)
-	)
-	(wire
-		(pts
-			(xy 73.66 93.98) (xy 87.63 93.98)
-		)
-		(stroke
-			(width 0)
-			(type default)
-		)
-	)
-	(wire
-		(pts
-			(xy 165.1 82.55) (xy 220.98 82.55)
-		)
-		(stroke
-			(width 0)
-			(type default)
-		)
-	)
-	(wire
-		(pts
-			(xy 165.1 73.66) (xy 220.98 73.66)
 		)
 		(stroke
@@
 			)
 		)
-		(pin "LIDAR_USART2_TX" input
-			(at 165.1 71.12 0)
-			(effects
-				(font
-					(size 1.27 1.27)
-				)
-				(justify right)
-			)
-		)
 		(pin "Bluetooth_USART3_RX" input
 			(at 165.1 80.01 0)
@@
 		)
 		(pin "M_CTR" input
-			(at 165.1 73.66 0)
+			(at 165.1 71.12 0)
 			(effects
 				(font
@@
 			)
 		)
-		(pin "LIDAR_USART2_TX" input
-			(at 220.98 71.12 180)
-			(effects
-				(font
-					(size 1.27 1.27)
-				)
-				(justify left)
-			)
-		)
 		(pin "Bluetooth_USART3_RX" input
 			(at 220.98 80.01 180)
@@
 		)
 		(pin "M_CTR" input
-			(at 220.98 73.66 180)
-			(effects
-				(font
+			(at 220.98 71.12 180)
+			(effects
+				(font
