File: Hardware/KiCad/Projet_Robot.kicad_sch (KiCad schematic)
At the start: 0 parts

Commit message: e
Other:
- sheet Capteurs ports: added Bluetooth_En; removed none
- sheet µcontrolleur ports: added Bluetooth_En; removed none
Changed lines of the file:
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@@
+	(wire
+		(pts
+			(xy 165.1 85.09) (xy 220.98 85.09)
+		)
+		(stroke
+			(width 0)
+			(type default)
+		)
+	)
 	(wire
 		(pts
@@
 			)
 		)
+		(pin "Bluetooth_En" input
+			(at 165.1 85.09 0)
+			(effects
+				(font
+					(size 1.27 1.27)
+				)
+				(justify right)
+			)
+		)
 		(instances
 			(project "Projet_Robot"
@@
 			(effects
 				(font
+					(size 1.27 1.27)
+				)
+				(justify left)
+			)
+		)
+		(pin "Bluetooth_En" input
+			(at 220.98 85.09 180)
+			(effects
+				(font

Commit message: gerbers
Other:
- company: (none) -> Ensea
- title: (none) -> Hello_kitty
Changed lines of the file:
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@@
 	(generator_version "9.0")
 	(paper "A4")
+	(title_block
+		(title "Hello_kitty")
+		(date "2025-10-13")
+		(company "Ensea")
+		(comment 1 "Aymen_BEN_JEMAA")
+		(comment 2 "Ezer_SOLTANI")
+		(comment 3 "Serine_ROUABAH")
+	)
 	(wire
 		(pts
