File: Hardware/KiCad/Projet_Robot.kicad_pcb (KiCad board)
At the start: 4 copper layers, 78 parts, among them IC1 ADXL343BCCZ-RL, IC2 MP1475DJ-LF-P, J11 Conn_ST_STDC14, J2 Conn_01x06, J201 Conn_01x06, J3 Conn_01x06, J4 Conn_01x06, J5 Conn_01x05, J6 Conn_01x06, J7 Conn_01x06, J8 Conn_01x02, SW1 SW_Push, SW2 Wurth 472121020311, SW3 SW_Push, U1 STM32G431CBUx, U2 ZXBM5210-SP, U3 ZXBM5210-SP, Y1 16MHz

Commit message: s
Parts:
- J7: footprint Connector_JST:JST_XH_B6B-XH-AM_1x06_P2.50mm_Vertical -> Connector_JST:JST_XH_B6B-XH-A_1x06_P2.50mm_Vertical
- moved J3 173.7 mm to (196.8, 52.5)
- moved J11 141.8 mm to (204.3, 68.1)
- moved H1 4.43 mm to (180.0, 50.0)
- moved H2 3.94 mm to (230.0, 50.0)
- moved H3 2.81 mm to (180.0, 99.0)
- moved H4 1.16 mm to (230.0, 99.0)
Other:
- board outline added: 58 x 57 mm
Changed lines of the file:
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@@
 	(footprint "Connector_JST:JST_XH_B6B-XH-AM_1x06_P2.50mm_Vertical"
 		(layer "F.Cu")
-		(at 23.865 36.5)
+		(at 196.85 52.55)
 		(descr "JST XH series connector, B6B-XH-AM, with boss (http://www.jst-mfg.com/product/pdf/eng/eXH.pdf), generated with kicad-footprint-generator")
 		(tags "connector JST XH vertical boss")
@@
 	(footprint "MountingHole:MountingHole_3.2mm_M3_Pad_Via"
 		(layer "F.Cu")
-		(at 182.647056 53.552944)
+		(at 180 50)
 		(descr "Mounting Hole 3.2mm, M3, generated by kicad-footprint-generator mountinghole.py")
 		(tags "mountinghole M3")
@@
 	(footprint "MountingHole:MountingHole_3.2mm_M3_Pad_Via"
 		(layer "F.Cu")
-		(at 231.2 53.75)
+		(at 230 50)
 		(descr "Mounting Hole 3.2mm, M3, generated by kicad-footprint-generator mountinghole.py")
 		(tags "mountinghole M3")
@@
 	(footprint "MountingHole:MountingHole_3.2mm_M3_Pad_Via"
 		(layer "F.Cu")
-		(at 230.977944 99.627944)
+		(at 230 99)
 		(descr "Mounting Hole 3.2mm, M3, generated by kicad-footprint-generator mountinghole.py")
 		(tags "mountinghole M3")
@@
 	(footprint "Connector_PinHeader_1.27mm:PinHeader_2x07_P1.27mm_Vertical_SMD"
 		(layer "F.Cu")
-		(at 63.235 53.66)
+		(at 204.3 68.09)
 		(descr "surface-mounted straight pin header, 2x07, 1.27mm pitch, double rows")
 		(tags "Surface mounted pin header SMD 2x07 1.27mm double row")
@@
 		)
 	)
-	(footprint "Connector_JST:JST_XH_B6B-XH-AM_1x06_P2.50mm_Vertical"
+	(footprint "Connector_JST:JST_XH_B6B-XH-A_1x06_P2.50mm_Vertical"
 		(layer "F.Cu")
 		(at 23.865 67.7)
-		(descr "JST XH series connector, B6B-XH-AM, with boss (http://www.jst-mfg.com/product/pdf/eng/eXH.pdf), generated with kicad-footprint-generator")
-		(tags "connector JST XH vertical boss")
+		(descr "JST XH series connector, B6B-XH-A (http://www.jst-mfg.com/product/pdf/eng/eXH.pdf), generated with kicad-footprint-generator")
+		(tags "connector JST XH vertical")
 		(property "Reference" "J7"
 			(at 6.25 -3.55 0)
@@
 		(fp_line
 			(start -1.8 -0.2)
-			(end -1.8 1.14)
+			(end -1.8 2.75)
+			(stroke
+				(width 0.12)
+				(type solid)
+			)
+			(layer "F.SilkS")
+		)
+		(fp_line
+			(start -1.8 2.75)
+			(end 6.25 2.75)
 			(stroke
 				(width 0.12)
@@
 		)
 		(fp_line
-			(start 6.25 2.75)
-			(end -0.74 2.75)
-			(stroke
-				(width 0.12)
-				(type solid)
-			)
-			(layer "F.SilkS")
-		)
-		(fp_line
 			(start 11.75 -2.45)
 			(end 0.75 -2.45)
@@
 			)
 		)
-		(pad "" np_thru_hole circle
-			(at -1.6 2)
-			(size 1.2 1.2)
-			(drill 1.2)
-			(layers "*.Cu" "*.Mask")
-		)
 		(pad "1" thru_hole roundrect
 			(at 0 0)
@@
 		)
 		(embedded_fonts no)
-		(model "${KICAD9_3DMODEL_DIR}/Connector_JST.3dshapes/JST_XH_B6B-XH-AM_1x06_P2.50mm_Vertical.step"
+		(model "${KICAD9_3DMODEL_DIR}/Connector_JST.3dshapes/JST_XH_B6B-XH-A_1x06_P2.50mm_Vertical.step"
 			(offset
 				(xyz 0 0 0)
@@
 	(footprint "MountingHole:MountingHole_3.2mm_M3_Pad_Via"
 		(layer "F.Cu")
-		(at 182.675 99.85)
+		(at 180 99)
 		(descr "Mounting Hole 3.2mm, M3, generated by kicad-footprint-generator mountinghole.py")
 		(tags "mountinghole M3")
@@
 		)
 	)
+	(gr_arc
+		(start 230 46)
+		(mid 232.828427 47.171573)
+		(end 234 50)
+		(stroke
+			(width 0.05)
+			(type default)
+		)
+		(layer "Edge.Cuts")
+	)
 	(gr_line
-		(start 231.052944 103.802944)
-		(end 182.575002 103.875)
+		(start 180 46)
+		(end 230 46)
 		(stroke
-			(width 0.2)
+			(width 0.05)
 			(type default)
 		)
-		(layer "F.Cu")
+		(layer "Edge.Cuts")
 	)
 	(gr_arc
-		(start 235.153618 99.627944)
-		(mid 233.95699 102.553955)
-		(end 231.052944 103.802944)
+		(start 176 50)
+		(mid 177.171573 47.171573)
+		(end 180 46)
 		(stroke
-			(width 0.2)
+			(width 0.05)
 			(type default)
 		)
-		(layer "F.Cu")
+		(layer "Edge.Cuts")
 	)
 	(gr_line
-		(start 235.33 53.75)
-		(end 235.153618 99.627944)
+		(start 234 50)
+		(end 234 99)
 		(stroke
-			(width 0.2)
+			(width 0.05)
 			(type default)
 		)
-		(layer "F.Cu")
+		(layer "Edge.Cuts")
 	)
 	(gr_line
-		(start 231.25 49.6)
-		(end 182.620941 49.62)
+		(start 180 103)
+		(end 230 103)
 		(stroke
-			(width 0.2)
+			(width 0.05)
 			(type default)
 		)
-		(layer "F.Cu")
+		(layer "Edge.Cuts")
 	)
 	(gr_arc
-		(start 231.2 49.62)
-		(mid 234.120351 50.829649)
-		(end 235.33 53.75)
+		(start 180 103)
+		(mid 177.171573 101.828427)
+		(end 176 99)
 		(stroke
-			(width 0.2)
+			(width 0.05)
 			(type default)
 		)
-		(layer "F.Cu")
+		(layer "Edge.Cuts")
 	)
 	(gr_arc
-		(start 178.714201 53.526443)
-		(mid 179.87543 50.762579)
-		(end 182.647056 49.62)
+		(start 234 99)
+		(mid 232.828427 101.828427)
+		(end 230 103)
 		(stroke
-			(width 0.2)
+			(width 0.05)
 			(type default)
 		)
-		(layer "F.Cu")
+		(layer "Edge.Cuts")
 	)
 	(gr_line
-		(start 178.714201 53.579209)
-		(end 178.648758 99.85)
+		(start 176 99)
+		(end 176 50)
 		(stroke
-			(width 0.2)
+			(width 0.05)
 			(type default)
 		)
-		(layer "F.Cu")
-	)
-	(gr_arc
-		(start 182.775 103.875)
-		(mid 179.863595 102.732122)
-		(end 178.648758 99.85)
-		(stroke
-			(width 0.2)
-			(type default)
-		)
-		(layer "F.Cu")
+		(layer "Edge.Cuts")
 	)
 	(embedded_fonts no)

Commit message: hhhh
Parts:
- added C27: 1u, Capacitor_SMD:C_0201_0603Metric, F.Cu at (101.0, 39.9)
- added C28: 1u, Capacitor_SMD:C_0201_0603Metric, F.Cu at (101.0, 41.6)
- added C29: 1u, Capacitor_SMD:C_0201_0603Metric, F.Cu at (101.0, 43.4)
- added C30: 1u, Capacitor_SMD:C_0201_0603Metric, F.Cu at (101.0, 45.1)
- added C31: 1u, Capacitor_SMD:C_0201_0603Metric, F.Cu at (101.0, 46.9)
- added C32: 100nf, Capacitor_SMD:C_0201_0603Metric, F.Cu at (109.5, 39.9)
- added R17: 10k, Resistor_SMD:R_0603_1608Metric, F.Cu at (106.2, 40.3)
- added R20: 10K, Resistor_SMD:R_0603_1608Metric, F.Cu at (106.2, 42.8)
- added TP5: TestPoint, TestPoint:TestPoint_Pad_D1.5mm, F.Cu at (98.0, 40.8)
- added TP6: TestPoint, TestPoint:TestPoint_Pad_D1.5mm, F.Cu at (98.0, 44.4)
- added TP7: TestPoint, TestPoint:TestPoint_Pad_D1.5mm, F.Cu at (98.0, 47.9)
- added TP8: TestPoint, TestPoint:TestPoint_Pad_D1.5mm, F.Cu at (98.0, 51.5)
- added TP9: TestPoint, TestPoint:TestPoint_Pad_D1.5mm, F.Cu at (98.0, 55.0)
- J3, J4, J5, J6: footprint Connector_JST:JST_XH_B6B-XH-AM_1x06_P2.50mm_Vertical -> Connector_JST:JST_XH_B6B-XH-A_1x06_P2.50mm_Vertical
Connections:
- SW3 pad 1: /µcontrolleur/BOUTON_Chat/Souris -> Net-(R17-Pad2)

Commit message: s
s
Parts:
- removed J5: Conn_01x05, Connector_JST:JST_XH_B6B-XH-A_1x06_P2.50mm_Vertical
- added J1: Conn_01x05, Connector_JST:JST_XH_B5B-XH-A_1x05_P2.50mm_Vertical, F.Cu at (121.0, 74.5)
- added J9: Conn_01x06, Connector_PinSocket_2.54mm:PinSocket_1x06_P2.54mm_Vertical, F.Cu at (115.2, 73.5)
- added PS1: BU33SD5WG-TR, Package_SO:TSOP-5_1.65x3.05mm_P0.95mm, F.Cu at (42.8, 108.0)
- H1, H2, H3, H4: value MountingHole -> MountingHole_Pad; footprint MountingHole:MountingHole_3.2mm_M3_Pad_Via -> MountingHole:MountingHole_3.2mm_M3_ISO7380_Pad
- L2: footprint Resistor_SMD:R_0603_1608Metric -> Inductor_SMD:L_APV_ANR5040
- moved U1 134.1 mm to (205.0, 75.0)
- moved H1 85.5 mm to (262.0, 74.2)
- moved H3 82.6 mm to (262.0, 88.8)
- moved H2 44.9 mm to (262.0, 81.5)
- moved H4 32.1 mm to (262.0, 96.0)
- moved J11 24.5 mm to (228.1, 74.2), turned to 180 degrees
- moved L2 13.1 mm to (51.0, 62.0)
Connections:
- H1 pad 1: (no net) -> GND
- H2 pad 1: (no net) -> GND
- H3 pad 1: (no net) -> GND
- H4 pad 1: (no net) -> GND
Routing:
- added copper zone on In1.Cu, net GND

Commit message: w
Parts:
- H1, H2, H3, H4: footprint MountingHole:MountingHole_3.2mm_M3_ISO7380_Pad -> MountingHole:MountingHole_3.2mm_M3_Pad_Via
- moved TOF2 190.2 mm to (206.0, 99.0)
- moved TOF3 176.6 mm to (187.0, 127.5), turned to 90 degrees
- moved BT1 166.5 mm to (215.0, 50.0), turned to 180 degrees
- moved Motor2 155.4 mm to (178.0, 58.0), turned to -90 degrees
- moved B-Res1 131.3 mm to (203.0, 50.0)
- moved ch/sou1 117.8 mm to (190.0, 50.0), turned to 180 degrees
- moved Lidar1 111.2 mm to (231.0, 58.0), turned to -90 degrees
- moved Motor1 106.4 mm to (178.0, 76.5), turned to -90 degrees
- moved H1 85.5 mm to (180.0, 50.0)
- moved H3 82.6 mm to (180.0, 99.0)
- moved TOF1 47.5 mm to (187.0, 99.0)
- moved H2 44.9 mm to (230.0, 50.0)
- moved alim_batt1 40.1 mm to (98.5, 73.0)
- moved H4 32.1 mm to (230.0, 99.0)
- moved J11 3.02 mm to (229.9, 76.5)
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- renumbered SW1 to B-Res1, J9 to Bluetooth1, J1 to Lidar1, J201 to Motor1, J2 to Motor2, J3 to TOF1, J4 to TOF2, J6 to TOF3, J7 to TOF4, J8 to alim_batt1, SW2 to batterie1, SW3 to ch/sou1

Commit message: s
Parts:
- alim_batt1: value Conn_01x02 -> alim
- moved batterie1 175.0 mm to (222.2, 57.9), turned to 90 degrees
- moved M2 162.4 mm to (185.5, 70.9)
- moved PS1 142.0 mm to (183.8, 91.5)
- moved alim_batt1 125.4 mm to (222.0, 51.5), turned to 90 degrees
- moved TOF4 115.9 mm to (139.5, 76.0)
- moved M1 113.4 mm to (185.5, 77.0), turned to 180 degrees
- moved Bluetooth1 109.8 mm to (224.0, 88.3)
- moved TOF3 76.0 mm to (139.5, 68.2), turned to 0 degrees
- moved R18 12.3 mm to (73.8, 90.9)
- moved TP1 12.3 mm to (70.0, 91.5)
- moved TP2 12.3 mm to (70.0, 95.0)
- moved IC2 12.3 mm to (50.4, 97.0)
- moved C23 12.3 mm to (77.0, 90.5)
- moved C24 12.3 mm to (77.0, 92.3)
- moved R19 12.3 mm to (73.8, 93.4)
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- renumbered U3 to M1, U2 to M2

Commit message: q
Parts:
- IC2: footprint Package_TO_SOT_SMD:TSOT-23 -> Package_TO_SOT_SMD:TSOT-23-8_HandSoldering
- alim_batt1: value alim -> Conn_01x02
- moved L2 167.7 mm to (216.8, 87.4)
- moved IC2 166.5 mm to (214.1, 66.7)
- moved C17 160.1 mm to (224.9, 83.2)
- moved C18 160.1 mm to (224.9, 85.0)
- moved C19 160.1 mm to (224.9, 86.7)
- moved C20 160.1 mm to (224.9, 88.5)
- moved R13 157.1 mm to (218.7, 69.7)
- moved R7 154.7 mm to (212.4, 69.7)
- moved R8 154.6 mm to (212.3, 71.4)
- moved IC1 154.0 mm to (196.0, 37.7)
- moved R12 153.7 mm to (215.5, 73.5)
- moved R11 153.7 mm to (215.5, 71.4)
- moved R10 153.6 mm to (215.5, 69.7)
- moved C13 153.2 mm to (210.8, 62.0)
- moved C12 153.0 mm to (210.8, 63.6)
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Routing:
- net GND: track 0.00 -> 51.3 mm
- net /Capteurs/TOF3_XSHUT: track 0.00 -> 32.4 mm
- net /Capteurs/tof3_GPIO: track 0.00 -> 27.1 mm, vias 0 -> 2
- net /Capteurs/TOF4_XSHUT: track 0.00 -> 25.2 mm
- net /Capteurs/TOF2_XSHUT: track 0.00 -> 23.6 mm
- net /Capteurs/TOF1_XSHUT: track 0.00 -> 15.0 mm
- net /Capteurs/I2C1_SDA: track 0.00 -> 14.0 mm
- net /Capteurs/I2C1_SCL: track 0.00 -> 14.0 mm

Commit message: 1
Routing:
- net /Capteurs/tof2_GPIO: track 0.00 -> 25.3 mm, vias 0 -> 2
- net /Capteurs/tof4_GPIO: track 0.00 -> 20.1 mm, vias 0 -> 2
- net /Capteurs/tof1_GPIO: track 0.00 -> 17.8 mm, vias 0 -> 2
- net /Capteurs/TOF4_XSHUT: track 25.2 -> 26.0 mm
- net /Capteurs/TOF3_XSHUT: track 32.4 -> 33.1 mm
