File: Hardware/KiCad/Projet_Robot.kicad_pcb (KiCad board)
At the start: 4 copper layers, 58 x 57 mm, 93 parts, among them IC1 ADXL343BCCZ-RL, IC2 MP1475DJ-LF-P, J11 Conn_ST_STDC14, M1 ZXBM5210-SP, M2 ZXBM5210-SP, U1 STM32G431CBUx, Y1 16MHz

Commit message: s
Parts:
- moved alim_batt1 31.6 mm to (250.0, 90.0)
- moved J11 19.5 mm to (249.3, 74.3)
- moved C17 18.4 mm to (206.4, 82.2)
- moved C18 18.4 mm to (206.4, 83.9)
- moved C19 18.4 mm to (206.4, 85.7)
- moved C20 18.4 mm to (206.4, 87.4)
- moved Lidar1 16.9 mm to (226.9, 74.4)
- moved Bluetooth1 9.39 mm to (227.9, 56.0)
- moved H2 4.00 mm to (226.0, 50.0)
- moved H4 4.00 mm to (226.0, 99.0)
Routing:
- net GND: track 51.3 -> 46.4 mm
Other:
- board size 58 x 57 mm -> 54.1 x 57 mm
Changed lines of the file:
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@@
 	(footprint "Connector_PinSocket_2.54mm:PinSocket_1x06_P2.54mm_Vertical"
 		(layer "F.Cu")
-		(at 223.3 47.8)
+		(at 227.92 55.97)
 		(descr "Through hole straight socket strip, 1x06, 2.54mm pitch, single row (from Kicad 4.0.7), script generated")
 		(tags "Through hole socket strip THT 1x06 2.54mm single row")
@@
 		)
 		(fp_text user "${REFERENCE}"
-			(at 0 0 90)
+			(at -9.9 0 90)
 			(layer "F.Fab")
 			(effects
@@
 	(footprint "Connector_JST:JST_XH_B5B-XH-A_1x05_P2.50mm_Vertical"
 		(layer "F.Cu")
-		(at 231 58 -90)
+		(at 226.93 74.44 -90)
 		(descr "JST XH series connector, B5B-XH-A (http://www.jst-mfg.com/product/pdf/eng/eXH.pdf), generated with kicad-footprint-generator")
 		(tags "connector JST XH vertical")
@@
 	(footprint "Capacitor_SMD:C_0201_0603Metric"
 		(layer "F.Cu")
-		(at 224.855 84.95)
+		(at 206.435 83.9)
 		(descr "Capacitor SMD 0201 (0603 Metric), square (rectangular) end terminal, IPC-7351 nominal, (Body size source: https://www.vishay.com/docs/20052/crcw0201e3.pdf), generated with kicad-footprint-generator")
 		(tags "capacitor")
@@
 	(footprint "Connector_JST:JST_EH_B2B-EH-A_1x02_P2.50mm_Vertical"
 		(layer "F.Cu")
-		(at 220 100)
+		(at 250 90)
 		(descr "JST EH series connector, B2B-EH-A (http://www.jst-mfg.com/product/pdf/eng/eEH.pdf), generated with kicad-footprint-generator")
 		(tags "connector JST EH vertical")
@@
 	(footprint "MountingHole:MountingHole_3.2mm_M3_Pad_Via"
 		(layer "F.Cu")
-		(at 230 50)
+		(at 226 50)
 		(descr "Mounting Hole 3.2mm, M3, generated by kicad-footprint-generator mountinghole.py")
 		(tags "mountinghole M3")
@@
 	(footprint "Capacitor_SMD:C_0201_0603Metric"
 		(layer "F.Cu")
-		(at 224.855 83.2)
+		(at 206.435 82.15)
 		(descr "Capacitor SMD 0201 (0603 Metric), square (rectangular) end terminal, IPC-7351 nominal, (Body size source: https://www.vishay.com/docs/20052/crcw0201e3.pdf), generated with kicad-footprint-generator")
 		(tags "capacitor")
@@
 	(footprint "MountingHole:MountingHole_3.2mm_M3_Pad_Via"
 		(layer "F.Cu")
-		(at 230 99)
+		(at 226 99)
 		(descr "Mounting Hole 3.2mm, M3, generated by kicad-footprint-generator mountinghole.py")
 		(tags "mountinghole M3")
@@
 			(at 0 4.15 0)
 			(layer "F.Fab")
+			(hide yes)
 			(effects
 				(font
@@
 	(footprint "Connector_PinHeader_1.27mm:PinHeader_2x07_P1.27mm_Vertical_SMD"
 		(layer "F.Cu")
-		(at 229.95 76.54 180)
+		(at 249.35 74.26 180)
 		(descr "surface-mounted straight pin header, 2x07, 1.27mm pitch, double rows")
 		(tags "Surface mounted pin header SMD 2x07 1.27mm double row")
@@
 	(footprint "Capacitor_SMD:C_0201_0603Metric"
 		(layer "F.Cu")
-		(at 224.855 88.45)
+		(at 206.435 87.4)
 		(descr "Capacitor SMD 0201 (0603 Metric), square (rectangular) end terminal, IPC-7351 nominal, (Body size source: https://www.vishay.com/docs/20052/crcw0201e3.pdf), generated with kicad-footprint-generator")
 		(tags "capacitor")
@@
 	(footprint "Capacitor_SMD:C_0201_0603Metric"
 		(layer "F.Cu")
-		(at 224.855 86.7)
+		(at 206.435 85.65)
 		(descr "Capacitor SMD 0201 (0603 Metric), square (rectangular) end terminal, IPC-7351 nominal, (Body size source: https://www.vishay.com/docs/20052/crcw0201e3.pdf), generated with kicad-footprint-generator")
 		(tags "capacitor")
@@
 	)
 	(gr_arc
-		(start 230 46)
-		(mid 232.828427 47.171573)
-		(end 234 50)
+		(start 226.121573 46)
+		(mid 228.95 47.171573)
+		(end 230.121573 50)
 		(stroke
 			(width 0.05)
@@
 	(gr_line
 		(start 180 46)
-		(end 230 46)
+		(end 226.121573 46)
 		(stroke
 			(width 0.05)
@@
 	)
 	(gr_line
-		(start 234 50)
-		(end 234 99)
+		(start 230.121573 50)
+		(end 230 99)
 		(stroke
 			(width 0.05)
@@
 	(gr_line
 		(start 180 103)
-		(end 230 103)
+		(end 225.94177 103.04)
 		(stroke
 			(width 0.05)
@@
 	)
 	(gr_arc
-		(start 234 99)
-		(mid 232.828427 101.828427)
-		(end 230 103)
+		(start 230.004617 98.965383)
+		(mid 228.811189 101.846572)
+		(end 225.93 103.04)
 		(stroke
 			(width 0.05)
@@
 		(width 0.1)
 		(layer "F.Cu")
-		(net 2)
-	)
-	(segment
-		(start 230 50)
-		(end 226.551 46.551)
-		(width 0.1)
-		(layer "F.Cu")

Commit message: M
Parts:
- moved ch/sou1 67.6 mm to (186.5, 84.0), turned to -90 degrees
- moved B-Res1 60.2 mm to (195.2, 83.5), turned to 90 degrees
- moved M1 4.43 mm to (186.0, 72.6)
- moved M2 4.43 mm to (186.0, 66.5)
- moved PS1 4.12 mm to (191.5, 66.0)
- moved Y1 3.36 mm to (192.5, 72.0), turned to 90 degrees

Commit message: A
Parts:
- moved C14 74.4 mm to (209.8, 84.0)
- moved D4 69.5 mm to (190.7, 96.0)
- moved C15 68.4 mm to (213.2, 84.0)
- moved R6 57.2 mm to (190.7, 93.0)
- moved C22 47.9 mm to (157.7, 161.0)
- moved C25 47.9 mm to (157.7, 162.8)
- moved IC1 45.3 mm to (205.5, 82.0)
- moved J11 45.0 mm to (211.5, 98.5), turned to 90 degrees
- moved C20 30.1 mm to (221.8, 61.5)
- moved C19 28.3 mm to (224.0, 63.5)
- moved L2 28.0 mm to (203.2, 63.0)
- moved C18 23.3 mm to (212.8, 61.5)
- moved alim_batt1 22.9 mm to (227.2, 92.5), turned to 90 degrees
- moved C17 21.6 mm to (217.3, 63.5)
- moved C13 18.1 mm to (219.7, 77.8)
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Routing:
- net +5V: track 0.00 -> 1.67 mm, vias 0 -> 1
- net GND: track 46.4 -> 47.3 mm

Commit message: s
Parts:
- moved R8 38.5 mm to (248.9, 82.8)
- moved R12 31.0 mm to (243.6, 70.2)
- moved C17 30.1 mm to (244.4, 76.7)
- moved C18 30.1 mm to (239.9, 74.7)
- moved R7 30.1 mm to (240.2, 78.2)
- moved R11 27.3 mm to (241.6, 72.5)
- moved R10 27.0 mm to (239.8, 68.9)
- moved C20 26.9 mm to (245.8, 73.7)
- moved C12 24.1 mm to (244.7, 80.2)
- moved C19 24.1 mm to (245.7, 74.0)
- moved J11 22.2 mm to (225.9, 81.6), turned to 180 degrees
- moved C13 11.3 mm to (218.2, 89.0)
- moved C16 11.3 mm to (215.2, 91.7)
- moved R13 11.3 mm to (215.9, 82.2)
- moved R9 11.3 mm to (212.2, 90.7)
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
Commit message: s
Parts:
- moved C31 77.7 mm to (222.5, 57.3)
- moved C30 77.1 mm to (222.6, 56.3)
- moved C28 76.6 mm to (222.6, 53.4)
- moved C29 76.4 mm to (222.6, 55.4)
- moved C27 74.5 mm to (222.6, 54.5)
- moved C20 34.0 mm to (211.9, 71.1)
- moved C19 32.2 mm to (213.7, 71.1)
- moved C17 31.3 mm to (213.9, 69.7), turned to 180 degrees
- moved R12 28.4 mm to (216.2, 62.8), turned to 180 degrees
- moved C18 28.2 mm to (212.1, 69.8)
- moved R11 26.4 mm to (216.3, 65.0)
- moved R10 23.7 mm to (216.2, 70.0)
- moved alim_batt1 3.60 mm to (223.7, 93.3)
- moved Lidar1 0.19 mm to (227.3, 63.6)

Commit message: 1
Parts:
- moved R16 119.6 mm to (184.7, 71.5)
- moved R15 119.6 mm to (184.7, 69.0)
- moved R18 96.4 mm to (195.2, 78.5)
- moved R19 96.4 mm to (195.2, 81.0)
- moved C23 76.5 mm to (186.2, 88.5)
- moved C24 76.5 mm to (186.2, 90.2)
- moved ch/sou1 30.2 mm to (213.8, 97.0)
- moved B-Res1 16.4 mm to (205.2, 96.5)
- moved M1 8.00 mm to (185.0, 82.5), turned to 0 degrees
- moved C13 3.99 mm to (216.8, 85.3)
- moved R9 3.99 mm to (210.8, 87.0)
- moved C16 3.99 mm to (213.8, 88.0)
- moved BT1 2.97 mm to (195.5, 100.5)
- moved L2 2.64 mm to (204.0, 65.5)
- moved TP9 0.56 mm to (198.0, 68.0)
Routing:
- net /Capteurs/TOF3_XSHUT: track 33.1 -> 6.68 mm
- net /Capteurs/TOF4_XSHUT: track 26.0 -> 0.00 mm
- net /Capteurs/tof3_GPIO: track 26.9 -> 1.50 mm, vias 2 -> 0
- net /Capteurs/tof4_GPIO: track 20.1 -> 0.00 mm, vias 2 -> 0
- net /Capteurs/TOF2_XSHUT: track 23.6 -> 4.47 mm
- net /Capteurs/tof2_GPIO: track 25.3 -> 10.1 mm, vias 2 -> 0
- net /Capteurs/tof1_GPIO: track 17.8 -> 2.70 mm, vias 2 -> 0
- net /Capteurs/TOF1_XSHUT: track 15.0 -> 2.81 mm

Commit message: s
Parts:
- moved R7 55.8 mm to (186.7, 94.3)
Changed lines of the file:
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@@
 			(at 0 -1.43 0)
 			(layer "F.SilkS")
+			(hide yes)
 			(effects
 				(font
@@
 			(at 0 1.43 0)
 			(layer "F.Fab")
+			(hide yes)
 			(effects
 				(font
@@
 			(at 0 -1.05 0)
 			(layer "F.SilkS")
+			(hide yes)
 			(effects
 				(font
@@
 		)
 		(property "Value" "1 uF"
-			(at 0 1.05 0)
+			(at -0.025 1.06 0)
 			(layer "F.Fab")
+			(hide yes)
 			(effects
 				(font
@@
 		)
 		(fp_text user "${REFERENCE}"
-			(at 0 -0.68 0)
+			(at 0.045 -0.33 0)
 			(layer "F.Fab")
 			(effects
@@
 			(at 0 -1.05 0)
 			(layer "F.SilkS")
+			(hide yes)
 			(effects
 				(font
@@
 			(at 0 1.05 0)
 			(layer "F.Fab")
+			(hide yes)
 			(effects
 				(font
@@
 		)
 		(fp_text user "${REFERENCE}"
-			(at 0 -0.68 0)
+			(at 0 -0.37 0)
 			(layer "F.Fab")
 			(effects
@@
 	(footprint "Resistor_SMD:R_0603_1608Metric"
 		(layer "F.Cu")
-		(at 240.21 78.21)
+		(at 186.74 94.27)
 		(descr "Resistor SMD 0603 (1608 Metric), square (rectangular) end terminal, IPC-7351 nominal, (Body size source: IPC-SM-782 page 72, https://www.pcb-3d.com/wordpress/wp-content/uploads/ipc-sm-782a_amendment_1_and_2.pdf), generated with kicad-footprint-generator")
 		(tags "resistor")
@@
 			(at 0 -1.5 0)
 			(layer "F.SilkS")
+			(hide yes)
 			(effects
 				(font
@@
 			(at 0 1.43 0)
 			(layer "F.Fab")
+			(hide yes)
 			(effects
 				(font
@@
 		)
 		(fp_text user "${REFERENCE}"
-			(at 1.475 5.8 0)
+			(at 0 0 0)
 			(layer "F.Fab")
 			(effects
@@
 			(at 0 -1.43 0)
 			(layer "F.SilkS")
+			(hide yes)
 			(effects
 				(font
@@
 			(at 0 1.43 0)
 			(layer "F.Fab")
+			(hide yes)
 			(effects
 				(font

Commit message: 1
Parts:
- moved C1 73.3 mm to (198.0, 80.5)
- moved C4 73.3 mm to (198.0, 88.0)
- moved C7 73.3 mm to (202.0, 80.5)
- moved C2 73.3 mm to (198.0, 83.0)
- moved C3 73.3 mm to (198.0, 85.5)
- moved C5 73.3 mm to (198.0, 90.5)
- moved C6 73.3 mm to (198.0, 93.0)
- moved C8 73.3 mm to (202.0, 83.0)
- moved R1 70.6 mm to (194.5, 80.5)
- moved R2 70.6 mm to (194.5, 83.0)
- moved L1 66.2 mm to (194.2, 87.5)
- moved C12 30.2 mm to (214.5, 80.0)
- moved PS1 24.1 mm to (210.3, 81.0)
- moved R19 16.5 mm to (182.8, 92.0)
- moved R18 16.0 mm to (182.7, 88.5)
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