File: Hardware/KiCad/Projet_Robot.kicad_pcb (KiCad board)
At the start: 4 copper layers, 54.1 x 57 mm, 91 parts, among them IC1 ADX, IC2 MP1, M1 ZXB, M2 ZXB, U1 STM, Y1 16MHz

Commit message: Y
Parts:
- moved C25 38.5 mm to (135.9, 108.8), turned to 90 degrees
- moved TP4 34.2 mm to (136.4, 110.6)
- moved R15 33.6 mm to (134.4, 96.2), turned to 90 degrees
- moved TP3 33.6 mm to (133.6, 110.7)
- moved R16 31.1 mm to (137.2, 99.6), turned to 90 degrees
- moved TP1 25.0 mm to (133.0, 91.4)
- moved C24 24.0 mm to (136.1, 89.3), turned to 90 degrees
- moved TP2 21.9 mm to (136.1, 91.4)
- moved C23 21.3 mm to (137.4, 89.2), turned to -90 degrees
- moved C22 19.4 mm to (137.2, 108.9), turned to -90 degrees
- moved C30 19.0 mm to (151.2, 122.1)
- moved R20 12.8 mm to (150.8, 105.2), turned to 180 degrees
- moved R17 11.6 mm to (150.8, 106.9), turned to 180 degrees
- moved C11 11.0 mm to (143.7, 84.5), turned to -90 degrees
- moved C32 10.1 mm to (150.0, 103.6)
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Routing:
- net /µcontrolleur/SWDIO: track 86.0 -> 0.00 mm
- net /µcontrolleur/SWCLK: track 83.1 -> 0.00 mm
- net /Capteurs/TOF3_XSHUT: track 71.5 -> 0.00 mm
- net /Capteurs/I2C1_SCL: track 67.7 -> 0.00 mm, vias 4 -> 0
- net /Capteurs/I2C1_SDA: track 67.3 -> 0.00 mm, vias 3 -> 0
- net /Capteurs/tof2_GPIO: track 56.8 -> 0.00 mm
- net /Capteurs/TOF4_XSHUT: track 39.7 -> 0.00 mm
- net /Capteurs/tof4_GPIO: track 33.7 -> 0.00 mm, vias 2 -> 0
- net /Moteur2/ENC1_PH1: track 28.0 -> 0.00 mm
- net /µcontrolleur/NRST: track 26.0 -> 0.00 mm
- net /Moteur1/PWM_Mot1_CH2: track 25.0 -> 0.00 mm
- net /Capteurs/TOF2_XSHUT: track 24.9 -> 0.00 mm
- net /Moteur2/ENC1_PH2: track 23.2 -> 0.00 mm
- net /Capteurs/tof1_GPIO: track 21.8 -> 0.00 mm, vias 2 -> 0
- net /Moteur2/PWM_Mot1_CH2: track 20.9 -> 0.00 mm, vias 2 -> 0
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
Commit message: W
Parts:
- moved R15 10.3 mm to (140.2, 104.7)
- moved C6 9.20 mm to (146.5, 97.6)
- moved C7 0.91 mm to (148.6, 90.4)
- moved C21 0.28 mm to (146.5, 93.0)
Changed lines of the file:
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@@
 	(footprint "Capacitor_SMD:C_0603_1608Metric"
 		(layer "F.Cu")
-		(at 147.74 90.21)
+		(at 148.625 90.4)
 		(descr "Capacitor SMD 0603 (1608 Metric), square (rectangular) end terminal, IPC-7351 nominal, (Body size source: IPC-SM-782 page 76, https://www.pcb-3d.com/wordpress/wp-content/uploads/ipc-sm-782a_amendment_1_and_2.pdf), generated with kicad-footprint-generator")
 		(tags "capacitor")
@@
 	(footprint "Resistor_SMD:R_0603_1608Metric"
 		(layer "F.Cu")
-		(at 134.4 96.2 90)
+		(at 140.2 104.6625 90)
 		(descr "Resistor SMD 0603 (1608 Metric), square (rectangular) end terminal, IPC-7351 nominal, (Body size source: IPC-SM-782 page 72, https://www.pcb-3d.com/wordpress/wp-content/uploads/ipc-sm-782a_amendment_1_and_2.pdf), generated with kicad-footprint-generator")
 		(tags "resistor")
@@
 	(footprint "Capacitor_SMD:C_0603_1608Metric"
 		(layer "F.Cu")
-		(at 147.645 88.47)
+		(at 146.525 97.6)
 		(descr "Capacitor SMD 0603 (1608 Metric), square (rectangular) end terminal, IPC-7351 nominal, (Body size source: IPC-SM-782 page 76, https://www.pcb-3d.com/wordpress/wp-content/uploads/ipc-sm-782a_amendment_1_and_2.pdf), generated with kicad-footprint-generator")
 		(tags "capacitor")
@@
 	(footprint "Capacitor_SMD:C_0603_1608Metric"
 		(layer "F.Cu")
-		(at 146.25 92.97)
+		(at 146.525 93)
 		(descr "Capacitor SMD 0603 (1608 Metric), square (rectangular) end terminal, IPC-7351 nominal, (Body size source: IPC-SM-782 page 76, https://www.pcb-3d.com/wordpress/wp-content/uploads/ipc-sm-782a_amendment_1_and_2.pdf), generated with kicad-footprint-generator")
 		(tags "capacitor")

Commit message: M
Parts:
- moved C2 16.3 mm to (157.8, 97.8)
- moved C5 16.2 mm to (157.8, 99.3)
- moved C4 15.3 mm to (168.6, 94.7)
- moved C3 13.5 mm to (162.6, 94.7)
- moved Y1 13.1 mm to (165.6, 95.0)
- moved D2 7.78 mm to (159.3, 87.2)
- moved D5 7.78 mm to (159.3, 88.7)
- moved R14 7.78 mm to (162.4, 88.7)
- moved R4 7.78 mm to (162.4, 87.2)
- moved B-Res1 7.34 mm to (165.2, 106.3)
- moved L1 4.45 mm to (148.6, 88.9), turned to 0 degrees
- moved D1 3.55 mm to (162.1, 72.9)
- moved R5 3.52 mm to (165.7, 72.9)
- moved TP6 3.50 mm to (161.2, 98.8)
- moved C1 3.37 mm to (157.8, 95.3)
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
Commit message: K
Parts:
- moved R1 1.20 mm to (156.8, 101.9)
- moved R2 0.20 mm to (154.3, 101.9)
Routing:
- net /Capteurs/I2C1_SCL: track 0.00 -> 55.6 mm, vias 0 -> 4
- net /Capteurs/I2C1_SDA: track 0.00 -> 54.5 mm, vias 0 -> 2
- net /Capteurs/TOF4_XSHUT: track 0.00 -> 32.5 mm, vias 0 -> 2
- net /Capteurs/tof4_GPIO: track 0.00 -> 27.4 mm
- net /Capteurs/tof2_GPIO: track 0.00 -> 26.7 mm
- net /Capteurs/TOF2_XSHUT: track 0.00 -> 25.9 mm, vias 0 -> 2
- net /Capteurs/TOF3_XSHUT: track 0.00 -> 25.5 mm, vias 0 -> 2
- net /Capteurs/tof1_GPIO: track 0.00 -> 23.2 mm
- net /Capteurs/tof3_GPIO: track 0.00 -> 19.8 mm
- net /Capteurs/TOF1_XSHUT: track 0.00 -> 17.9 mm, vias 0 -> 2

Commit message: I
Parts:
- turned R17 to 90 degrees
Routing:
- net /µcontrolleur/BOUTON_Chat/Souris: track 0.00 -> 17.3 mm
- net Net-(R17-Pad2): track 0.00 -> 7.16 mm
Changed lines of the file:
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@@
 	(footprint "Resistor_SMD:R_0603_1608Metric"
 		(layer "F.Cu")
-		(at 150 108.675 -90)
+		(at 150 108.675 90)
 		(descr "Resistor SMD 0603 (1608 Metric), square (rectangular) end terminal, IPC-7351 nominal, (Body size source: IPC-SM-782 page 72, https://www.pcb-3d.com/wordpress/wp-content/uploads/ipc-sm-782a_amendment_1_and_2.pdf), generated with kicad-footprint-generator")
 		(tags "resistor")
@@
 		(attr smd)
 		(fp_line
+			(start -0.237258 -0.5225)
+			(end 0.237258 -0.5225)
+			(stroke
+				(width 0.12)
+				(type solid)
+			)
+			(layer "F.SilkS")
+		)
+		(fp_line
 			(start -0.237258 0.5225)
 			(end 0.237258 0.5225)
@@
 		)
 		(fp_line
-			(start -0.237258 -0.5225)
-			(end 0.237258 -0.5225)
-			(stroke
-				(width 0.12)
-				(type solid)
-			)
-			(layer "F.SilkS")
+			(start 1.48 -0.73)
+			(end 1.48 0.73)
+			(stroke
+				(width 0.05)
+				(type solid)
+			)
+			(layer "F.CrtYd")
+		)
+		(fp_line
+			(start -1.48 -0.73)
+			(end 1.48 -0.73)
+			(stroke
+				(width 0.05)
+				(type solid)
+			)
+			(layer "F.CrtYd")
+		)
+		(fp_line
+			(start 1.48 0.73)
+			(end -1.48 0.73)
+			(stroke
+				(width 0.05)
+				(type solid)
+			)
+			(layer "F.CrtYd")
 		)
 		(fp_line
@@
 		)
 		(fp_line
-			(start 1.48 0.73)
-			(end -1.48 0.73)
-			(stroke
-				(width 0.05)
-				(type solid)
-			)
-			(layer "F.CrtYd")
-		)
-		(fp_line
-			(start -1.48 -0.73)
-			(end 1.48 -0.73)
-			(stroke
-				(width 0.05)
-				(type solid)
-			)
-			(layer "F.CrtYd")
-		)
-		(fp_line
-			(start 1.48 -0.73)
-			(end 1.48 0.73)
-			(stroke
-				(width 0.05)
-				(type solid)
-			)
-			(layer "F.CrtYd")
+			(start 0.8 -0.4125)
+			(end 0.8 0.4125)
+			(stroke
+				(width 0.1)
+				(type solid)
+			)
+			(layer "F.Fab")
+		)
+		(fp_line
+			(start -0.8 -0.4125)
+			(end 0.8 -0.4125)
+			(stroke
+				(width 0.1)
+				(type solid)
+			)
+			(layer "F.Fab")
+		)
+		(fp_line
+			(start 0.8 0.4125)
+			(end -0.8 0.4125)
+			(stroke
+				(width 0.1)
+				(type solid)
+			)
+			(layer "F.Fab")
 		)
 		(fp_line
@@
 			(layer "F.Fab")
 		)
-		(fp_line
-			(start 0.8 0.4125)
-			(end -0.8 0.4125)
-			(stroke
-				(width 0.1)
-				(type solid)
-			)
-			(layer "F.Fab")
-		)
-		(fp_line
-			(start -0.8 -0.4125)
-			(end 0.8 -0.4125)
-			(stroke
-				(width 0.1)
-				(type solid)
-			)
-			(layer "F.Fab")
-		)
-		(fp_line
-			(start 0.8 -0.4125)
-			(end 0.8 0.4125)
-			(stroke
-				(width 0.1)
-				(type solid)
-			)
-			(layer "F.Fab")
-		)
 		(fp_text user "${REFERENCE}"
 			(at 0 0 90)
@@
 		)
 		(pad "1" smd roundrect
-			(at -0.825 0 270)
+			(at -0.825 0 90)
 			(size 0.8 0.95)
 			(layers "F.Cu" "F.Mask" "F.Paste")
@@
 		)
 		(pad "2" smd roundrect
-			(at 0.825 0 270)
+			(at 0.825 0 90)
 			(size 0.8 0.95)
 			(layers "F.Cu" "F.Mask" "F.Paste")
@@
 		(net 43)
 	)
+	(segment
+		(start 145.3625 94.6625)
+		(end 148.7225 94.6625)
+		(width 0.1)
+		(layer "F.Cu")
+		(net 62)
+	)
+	(segment
+		(start 144.9 98.4)
+		(end 144.9 95.125)
+		(width 0.1)
+		(layer "F.Cu")
+		(net 62)
+	)
+	(segment
+		(start 145.1 98.6)
+		(end 144.9 98.4)
+		(width 0.1)
+		(layer "F.Cu")
+		(net 62)
+	)
+	(segment
+		(start 144.9 95.125)
+		(end 145.3625 94.6625)
+		(width 0.1)
+		(layer "F.Cu")
+		(net 62)
+	)
+	(segment
+		(start 148.8 104.3)
+		(end 148.8 100.5)
+		(width 0.1)
+		(layer "F.Cu")
+		(net 62)
+	)
+	(segment
+		(start 150 104.85)
+		(end 149.35 104.85)
+		(width 0.1)
+		(layer "F.Cu")
+		(net 62)
+	)
+	(segment
+		(start 146.9 98.6)
+		(end 145.1 98.6)
+		(width 0.1)
+		(layer "F.Cu")
+		(net 62)
+	)
+	(segment
+		(start 149.35 104.85)
+		(end 148.8 104.3)
+		(width 0.1)
+		(layer "F.Cu")
+		(net 62)
+	)
+	(segment
+		(start 148.8 100.5)
+		(end 146.9 98.6)
+		(width 0.1)
+		(layer "F.Cu")
+		(net 62)
+	)
+	(segment
+		(start 148.499 104.467352)
+		(end 150 105.968352)
+		(width 0.1)
+		(layer "F.Cu")
+		(net 77)
+	)
+	(segment
+		(start 148.005 102.105)
+		(end 148.499 102.599)
+		(width 0.1)
+		(layer "F.Cu")
+		(net 77)
+	)
+	(segment
+		(start 150 106.5)
+		(end 150 107.85)
+		(width 0.1)
+		(layer "F.Cu")
+		(net 77)
+	)
+	(segment
+		(start 147.42 102.105)
+		(end 148.005 102.105)
+		(width 0.1)
+		(layer "F.Cu")
+		(net 77)
+	)
+	(segment
+		(start 148.499 102.599)
+		(end 148.499 104.467352)
+		(width 0.1)
+		(layer "F.Cu")
+		(net 77)
+	)
+	(segment
+		(start 150 105.968352)
+		(end 150 106.5)
+		(width 0.1)
+		(layer "F.Cu")
+		(net 77)
+	)
 	(zone

Commit message: Z
Routing:
- net /µcontrolleur/NRST: track 0.00 -> 18.6 mm

Commit message: YYY
Parts:
- IC1: value ADX -> ADXL343BCCZ-RL
- IC2: value MP1 -> MP1475DJ-LF-P
- M1, M2: value ZXB -> ZXBM5210-SP
- PS1: value BU3 -> BU33SD5WG-TR
- R10: value 20 -> 20k
- U1: value STM -> STM32G431CBUx
- moved C21 16.0 mm to (161.8, 88.2), turned to -90 degrees
- moved TP6 15.0 mm to (156.4, 84.6)
- moved C1 9.36 mm to (167.0, 93.4)
- moved C8 9.29 mm to (160.2, 88.1), turned to 90 degrees
- moved B-Res1 9.14 mm to (174.2, 104.7)
- moved BT1 9.14 mm to (147.4, 69.2)
- moved C12 9.14 mm to (151.9, 77.1)
- moved C16 9.14 mm to (166.1, 80.1)
- moved C17 9.14 mm to (162.2, 84.0)
- moved C22 9.14 mm to (146.2, 107.3)
- moved C23 9.14 mm to (146.4, 87.6)
- moved C26 9.14 mm to (183.3, 79.8)
- moved C29 9.14 mm to (160.2, 114.1)
- moved C30 9.14 mm to (160.2, 120.5)
- moved C31 9.14 mm to (159.2, 76.3)
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- renumbered stlink to J11
Routing:
- net /Moteur1/ENC1_PH2: track 0.00 -> 47.3 mm, vias 0 -> 4
- net /µcontrolleur/VCP_RX: track 0.00 -> 45.0 mm, vias 0 -> 2
- net /Moteur1/ENC1_PH1: track 0.00 -> 40.4 mm
- net /µcontrolleur/VCP_TX: track 0.00 -> 35.6 mm, vias 0 -> 2
- net /µcontrolleur/SWDIO: track 0.00 -> 28.3 mm, vias 0 -> 2
- net /Moteur2/ENC1_PH1: track 0.00 -> 28.1 mm, vias 0 -> 2
- net /µcontrolleur/SWCLK: track 0.00 -> 25.8 mm, vias 0 -> 2
- net /Moteur2/ENC1_PH2: track 0.00 -> 23.2 mm, vias 0 -> 2
- net /µcontrolleur/STATUS_CHAT_LED: track 0.00 -> 19.1 mm, vias 0 -> 2
- net /µcontrolleur/STATUS_SOURIS_LED: track 0.00 -> 18.9 mm, vias 0 -> 2
- net Net-(U1-PF1): track 0.00 -> 16.5 mm, vias 0 -> 2
- net +3.3V: track 0.00 -> 11.9 mm
- net Net-(U1-PF0): track 0.00 -> 11.0 mm, vias 0 -> 2
- net Net-(IC1-RESERVED_1): track 0.00 -> 5.58 mm
- net /µcontrolleur/NRST: track 18.6 -> 24.0 mm
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