File: Hardware/KiCad/_autosave-Projet_Robot.kicad_pcb (KiCad board)
At the start: 4 copper layers, 54.1 x 57 mm, 91 parts, among them IC1 ADXL343BCCZ-RL, IC2 MP1475DJ-LF-P, J11 Conn_ST_STDC14, M1 ZXBM5210-SP, M2 ZXBM5210-SP, U1 STM32G431CBUx, Y1 16MHz

Commit message: AAAA
Parts:
- moved C1 0.19 mm to (167.0, 93.6)
Routing:
- net /Capteurs/M_CTR: track 0.00 -> 38.4 mm, vias 0 -> 2
- net /Capteurs/LIDAR_USART2_RX: track 0.00 -> 20.2 mm, vias 0 -> 2
- net /Capteurs/ACC_INT1: track 0.00 -> 13.9 mm, vias 0 -> 2
- net /Capteurs/ACC_INT2: track 0.00 -> 10.2 mm, vias 0 -> 2
- net /Moteur1/ENC1_PH1: track 40.8 -> 42.1 mm
- net /Moteur1/ENC1_PH2: track 47.4 -> 48.0 mm
- net /Capteurs/I2C1_SCL: track 87.8 -> 88.4 mm
