File: Hardware/KiCad/moteur1.kicad_sch (KiCad schematic)
At the start: 8 parts, among them J2 Conn_01x06, U2 ZXBM5210-SP

Commit message: 1
u
Parts:
- added R17: 4.7 k, symbol Device:R_Small
Changed lines of the file:
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@@
+	(symbol
+		(lib_id "Device:R_Small")
+		(at 95.25 140.97 0)
+		(unit 1)
+		(exclude_from_sim no)
+		(in_bom yes)
+		(on_board yes)
+		(dnp no)
+		(property "Reference" "R17"
+			(at 89.408 139.446 0)
+			(effects
+				(font
+					(size 1.016 1.016)
+				)
+				(justify left)
+			)
+		)
+		(property "Value" "4.7 k"
+			(at 88.646 141.478 0)
+			(effects
+				(font
+					(size 1.27 1.27)
+				)
+				(justify left)
+			)
+		)
+		(property "Footprint" ""
+			(at 95.25 140.97 0)
+			(effects
+				(font
+					(size 1.27 1.27)
+				)
+				(hide yes)
+			)
+		)
+		(property "Datasheet" "~"
+			(at 95.25 140.97 0)
+			(effects
+				(font
+					(size 1.27 1.27)
+				)
+				(hide yes)
+			)
+		)
+		(property "Description" "Resistor, small symbol"
+			(at 95.25 140.97 0)
+			(effects
+				(font
+					(size 1.27 1.27)
+				)
+				(hide yes)
+			)
+		)
+		(pin "1"
+		)
+		(pin "2"
+		)
+		(instances
+			(project "Projet_Robot"
+				(path "/21a14c86-6900-4d4b-9d91-6c59051d0f41/1388fddc-2e50-4e98-ba2d-1c17e87787d8"
+					(reference "R20")
+					(unit 1)
+				)
+				(path "/21a14c86-6900-4d4b-9d91-6c59051d0f41/aa5a4c0f-7d13-4543-a78f-f39351de5880"
+					(reference "R17")
+					(unit 1)
+				)
+			)
+		)
+	)
 	(symbol
 		(lib_id "Device:R_Small")

Commit message: c
Parts:
- C22, C25: footprint (none) -> Capacitor_SMD:C_0201_0603Metric
- R15, R16, R17: footprint (none) -> Resistor_SMD:R_0603_1608Metric
Changed lines of the file:
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@@
 			)
 		)
-		(property "Footprint" ""
+		(property "Footprint" "Capacitor_SMD:C_0201_0603Metric"
 			(at 111.76 68.58 0)
 			(effects
@@
 			)
 		)
-		(property "Footprint" ""
+		(property "Footprint" "Resistor_SMD:R_0603_1608Metric"
 			(at 100.33 71.12 0)
 			(effects
@@
 			)
 		)
-		(property "Footprint" ""
+		(property "Footprint" "Capacitor_SMD:C_0201_0603Metric"
 			(at 138.43 66.04 0)
 			(effects
@@
 			)
 		)
-		(property "Footprint" ""
+		(property "Footprint" "Resistor_SMD:R_0603_1608Metric"
 			(at 95.25 140.97 0)
 			(effects
@@
 			)
 		)
-		(property "Footprint" ""
+		(property "Footprint" "Resistor_SMD:R_0603_1608Metric"
 			(at 100.33 82.55 0)
 			(effects

Commit message: CubeMX
Parts:
- removed R17: 4.7 k, Resistor_SMD:R_0603_1608Metric, symbol Device:R_Small
Changed lines of the file:
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@@
-	(symbol
-		(lib_id "Device:R_Small")
-		(at 95.25 140.97 0)
-		(unit 1)
-		(exclude_from_sim no)
-		(in_bom yes)
-		(on_board yes)
-		(dnp no)
-		(property "Reference" "R17"
-			(at 89.408 139.446 0)
-			(effects
-				(font
-					(size 1.016 1.016)
-				)
-				(justify left)
-			)
-		)
-		(property "Value" "4.7 k"
-			(at 88.646 141.478 0)
-			(effects
-				(font
-					(size 1.27 1.27)
-				)
-				(justify left)
-			)
-		)
-		(property "Footprint" "Resistor_SMD:R_0603_1608Metric"
-			(at 95.25 140.97 0)
-			(effects
-				(font
-					(size 1.27 1.27)
-				)
-				(hide yes)
-			)
-		)
-		(property "Datasheet" "~"
-			(at 95.25 140.97 0)
-			(effects
-				(font
-					(size 1.27 1.27)
-				)
-				(hide yes)
-			)
-		)
-		(property "Description" "Resistor, small symbol"
-			(at 95.25 140.97 0)
-			(effects
-				(font
-					(size 1.27 1.27)
-				)
-				(hide yes)
-			)
-		)
-		(pin "1"
-		)
-		(pin "2"
-		)
-		(instances
-			(project "Projet_Robot"
-				(path "/21a14c86-6900-4d4b-9d91-6c59051d0f41/1388fddc-2e50-4e98-ba2d-1c17e87787d8"
-					(reference "R20")
-					(unit 1)
-				)
-				(path "/21a14c86-6900-4d4b-9d91-6c59051d0f41/aa5a4c0f-7d13-4543-a78f-f39351de5880"
-					(reference "R17")
-					(unit 1)
-				)
-			)
-		)
-	)
 	(symbol
 		(lib_id "Device:R_Small")

Commit message: j
Changed lines of the file:
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@@
 	(paper "A4")
+	(junction
+		(at 77.47 53.34)
+		(diameter 0)
+		(color 0 0 0 0)
+	)
 	(junction
 		(at 111.76 64.77)
@@
 	(wire
 		(pts
-			(xy 77.47 52.07) (xy 77.47 60.96)
-		)
-		(stroke
-			(width 0)
-			(type default)
-		)
-	)
-	(wire
-		(pts
 			(xy 107.95 81.28) (xy 116.84 81.28)
 		)
@@
 	(wire
 		(pts
+			(xy 77.47 53.34) (xy 77.47 60.96)
+		)
+		(stroke
+			(width 0)
+			(type default)
+		)
+	)
+	(wire
+		(pts
 			(xy 147.32 78.74) (xy 137.16 78.74)
 		)
@@
 		(pts
 			(xy 137.16 83.82) (xy 147.32 83.82)
+		)
+		(stroke
+			(width 0)
+			(type default)
+		)
+	)
+	(wire
+		(pts
+			(xy 77.47 53.34) (xy 77.47 52.07)
 		)
 		(stroke
@@
 					(unit 1)
 				)
+			)
+		)
+	)
+	(symbol
+		(lib_id "power:PWR_FLAG")
+		(at 77.47 53.34 90)
+		(unit 1)
+		(exclude_from_sim no)
+		(in_bom yes)
+		(on_board yes)
+		(dnp no)
+		(fields_autoplaced yes)
+		(property "Reference" "#FLG03"
+			(at 75.565 53.34 0)
+			(effects
+				(font
+					(size 1.27 1.27)
+				)
+				(hide yes)
+			)
+		)
+		(property "Value" "PWR_FLAG"
+			(at 73.66 53.3399 90)
+			(effects
+				(font
+					(size 1.27 1.27)
+				)
+				(justify left)
+			)
+		)
+		(property "Footprint" ""
+			(at 77.47 53.34 0)
+			(effects
+				(font
+					(size 1.27 1.27)
+				)
+				(hide yes)
+			)
+		)
+		(property "Datasheet" "~"
+			(at 77.47 53.34 0)
+			(effects
+				(font
+					(size 1.27 1.27)
+				)
+				(hide yes)
+			)
+		)
+		(property "Description" "Special symbol for telling ERC where power comes from"
+			(at 77.47 53.34 0)
+			(effects
+				(font
+					(size 1.27 1.27)
+				)
+				(hide yes)
+			)
+		)
+		(pin "1"
+		)
+		(instances
+			(project ""
+				(path "/21a14c86-6900-4d4b-9d91-6c59051d0f41/1388fddc-2e50-4e98-ba2d-1c17e87787d8"
+					(reference "#FLG05")
+					(unit 1)
+				)
+				(path "/21a14c86-6900-4d4b-9d91-6c59051d0f41/aa5a4c0f-7d13-4543-a78f-f39351de5880"
+					(reference "#FLG03")
+					(unit 1)
+				)

Commit message: P
Connections:
- net V_BATT renamed +VBAT
Changed lines of the file:
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@@
 	(paper "A4")
-	(junction
-		(at 77.47 53.34)
-		(diameter 0)
-		(color 0 0 0 0)
-	)
 	(junction
 		(at 111.76 64.77)
@@
 	)
 	(junction
-		(at 100.33 86.36)
-		(diameter 0)
-		(color 0 0 0 0)
-	)
-	(junction
 		(at 129.54 60.96)
 		(diameter 0)
@@
 	(wire
 		(pts
-			(xy 100.33 86.36) (xy 100.33 88.9)
+			(xy 100.33 85.09) (xy 100.33 88.9)
 		)
 		(stroke
@@
 	(wire
 		(pts
-			(xy 77.47 53.34) (xy 77.47 60.96)
+			(xy 100.33 58.42) (xy 100.33 60.96)
 		)
 		(stroke
@@
 	(wire
 		(pts
-			(xy 77.47 60.96) (xy 100.33 60.96)
-		)
-		(stroke
-			(width 0)
-			(type default)
-		)
-	)
-	(wire
-		(pts
 			(xy 111.76 64.77) (xy 111.76 66.04)
 		)
@@
 		(pts
 			(xy 137.16 83.82) (xy 147.32 83.82)
-		)
-		(stroke
-			(width 0)
-			(type default)
-		)
-	)
-	(wire
-		(pts
-			(xy 77.47 53.34) (xy 77.47 52.07)
-		)
-		(stroke
-			(width 0)
-			(type default)
-		)
-	)
-	(wire
-		(pts
-			(xy 100.33 85.09) (xy 100.33 86.36)
 		)
 		(stroke
@@
 	)
 	(symbol
+		(lib_id "power:+7.5V")
+		(at 100.33 58.42 0)
+		(unit 1)
+		(exclude_from_sim no)
+		(in_bom yes)
+		(on_board yes)
+		(dnp no)
+		(fields_autoplaced yes)
+		(property "Reference" "#PWR01"
+			(at 100.33 62.23 0)
+			(effects
+				(font
+					(size 1.27 1.27)
+				)
+				(hide yes)
+			)
+		)
+		(property "Value" "+VBAT"
+			(at 100.33 53.34 0)
+			(effects
+				(font
+					(size 1.27 1.27)
+				)
+			)
+		)
+		(property "Footprint" ""
+			(at 100.33 58.42 0)
+			(effects
+				(font
+					(size 1.27 1.27)
+				)
+				(hide yes)
+			)
+		)
+		(property "Datasheet" ""
+			(at 100.33 58.42 0)
+			(effects
+				(font
+					(size 1.27 1.27)
+				)
+				(hide yes)
+			)
+		)
+		(property "Description" "Power symbol creates a global label with name \"+7.5V\""
+			(at 100.33 58.42 0)
+			(effects
+				(font
+					(size 1.27 1.27)
+				)
+				(hide yes)
+			)
+		)
+		(pin "1"
+		)
+		(instances
+			(project ""
+				(path "/21a14c86-6900-4d4b-9d91-6c59051d0f41/1388fddc-2e50-4e98-ba2d-1c17e87787d8"
+					(reference "#PWR02")
+					(unit 1)
+				)
+				(path "/21a14c86-6900-4d4b-9d91-6c59051d0f41/aa5a4c0f-7d13-4543-a78f-f39351de5880"
+					(reference "#PWR01")
+					(unit 1)
+				)
+			)
+		)
+	)
+	(symbol
 		(lib_id "Device:C_Small")
 		(at 111.76 68.58 0)
@@
 	)
 	(symbol
-		(lib_id "power:+7.5V")
-		(at 77.47 52.07 0)
-		(unit 1)
-		(exclude_from_sim no)
-		(in_bom yes)
-		(on_board yes)
-		(dnp no)
-		(fields_autoplaced yes)
-		(property "Reference" "#PWR02"
-			(at 77.47 55.88 0)
-			(effects
-				(font
-					(size 1.27 1.27)
-				)
-				(hide yes)
-			)
-		)
-		(property "Value" "V_BATT"
-			(at 80.01 50.7999 0)
-			(effects
-				(font
-					(size 1.27 1.27)
-				)
-				(justify left)
-			)
-		)
-		(property "Footprint" ""
-			(at 77.47 52.07 0)
-			(effects
-				(font
-					(size 1.27 1.27)
-				)
-				(hide yes)
-			)
-		)
-		(property "Datasheet" ""
-			(at 77.47 52.07 0)
-			(effects
-				(font
-					(size 1.27 1.27)
-				)
-				(hide yes)
-			)
-		)
-		(property "Description" "Power symbol creates a global label with name \"+7.5V\""
-			(at 77.47 52.07 0)
-			(effects
-				(font
-					(size 1.27 1.27)
-				)
-				(hide yes)
-			)
-		)
-		(pin "1"
-		)
-		(instances
-			(project "Projet_Robot"
-				(path "/21a14c86-6900-4d4b-9d91-6c59051d0f41/1388fddc-2e50-4e98-ba2d-1c17e87787d8"
-					(reference "#PWR01")
-					(unit 1)
-				)
-				(path "/21a14c86-6900-4d4b-9d91-6c59051d0f41/aa5a4c0f-7d13-4543-a78f-f39351de5880"
-					(reference "#PWR02")
-					(unit 1)
-				)
-			)
-		)
-	)
-	(symbol
-		(lib_id "power:PWR_FLAG")
-		(at 77.47 53.34 90)
-		(unit 1)
-		(exclude_from_sim no)
-		(in_bom yes)
-		(on_board yes)
-		(dnp no)
-		(fields_autoplaced yes)
-		(property "Reference" "#FLG03"
-			(at 75.565 53.34 0)
-			(effects
-				(font
-					(size 1.27 1.27)
-				)
-				(hide yes)
-			)
-		)
-		(property "Value" "PWR_FLAG"
-			(at 73.66 53.3399 90)
-			(effects
-				(font
-					(size 1.27 1.27)
-				)
-				(justify left)
-			)
-		)
-		(property "Footprint" ""
-			(at 77.47 53.34 0)
-			(effects
-				(font
-					(size 1.27 1.27)
-				)
-				(hide yes)
-			)
-		)
-		(property "Datasheet" "~"
-			(at 77.47 53.34 0)
-			(effects
-				(font
-					(size 1.27 1.27)
-				)
-				(hide yes)
-			)
-		)
-		(property "Description" "Special symbol for telling ERC where power comes from"
-			(at 77.47 53.34 0)
-			(effects
-				(font
-					(size 1.27 1.27)
-				)
-				(hide yes)
-			)
-		)
-		(pin "1"
-		)
-		(instances
-			(project ""
-				(path "/21a14c86-6900-4d4b-9d91-6c59051d0f41/1388fddc-2e50-4e98-ba2d-1c17e87787d8"
-					(reference "#FLG05")
-					(unit 1)
-				)
-				(path "/21a14c86-6900-4d4b-9d91-6c59051d0f41/aa5a4c0f-7d13-4543-a78f-f39351de5880"
-					(reference "#FLG03")
-					(unit 1)
-				)
-			)
-		)
-	)
-	(symbol
 		(lib_id "Connector_Generic:Conn_01x06")
 		(at 199.39 82.55 0)
@@
 					(unit 1)
 				)
-			)
-		)
-	)
-	(symbol
-		(lib_id "power:PWR_FLAG")
-		(at 100.33 86.36 90)
-		(unit 1)
-		(exclude_from_sim no)
-		(in_bom yes)
-		(on_board yes)
-		(dnp no)
-		(fields_autoplaced yes)
-		(property "Reference" "#FLG02"
-			(at 98.425 86.36 0)
-			(effects
-				(font
-					(size 1.27 1.27)
-				)
-				(hide yes)
-			)
-		)
-		(property "Value" "PWR_FLAG"
-			(at 96.52 86.3599 90)
-			(effects
-				(font
-					(size 1.27 1.27)
-				)
-				(justify left)
-			)
-		)
-		(property "Footprint" ""
-			(at 100.33 86.36 0)
-			(effects
-				(font
-					(size 1.27 1.27)
-				)
-				(hide yes)
-			)
-		)
-		(property "Datasheet" "~"
-			(at 100.33 86.36 0)
-			(effects
-				(font
-					(size 1.27 1.27)
-				)
-				(hide yes)
-			)
-		)
-		(property "Description" "Special symbol for telling ERC where power comes from"
-			(at 100.33 86.36 0)
-			(effects
-				(font
-					(size 1.27 1.27)
-				)
-				(hide yes)
-			)
-		)
-		(pin "1"
-		)
-		(instances
-			(project "Projet_Robot"
-				(path "/21a14c86-6900-4d4b-9d91-6c59051d0f41/1388fddc-2e50-4e98-ba2d-1c17e87787d8"
-					(reference "#FLG06")
-					(unit 1)
-				)
-				(path "/21a14c86-6900-4d4b-9d91-6c59051d0f41/aa5a4c0f-7d13-4543-a78f-f39351de5880"
-					(reference "#FLG02")
-					(unit 1)
-				)

Commit message: w
Parts:
- renumbered J2 to Motor2
Changed lines of the file:
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@@
 		(dnp no)
 		(fields_autoplaced yes)
-		(property "Reference" "J2"
-			(at 201.93 82.55 0)
+		(property "Reference" "Motor2"
+			(at 201.93 83.8199 0)
 			(effects
 				(font
@@
 			(project "Projet_Robot"
 				(path "/21a14c86-6900-4d4b-9d91-6c59051d0f41/1388fddc-2e50-4e98-ba2d-1c17e87787d8"
-					(reference "J201")
+					(reference "Motor1")
 					(unit 1)
 				)
 				(path "/21a14c86-6900-4d4b-9d91-6c59051d0f41/aa5a4c0f-7d13-4543-a78f-f39351de5880"
-					(reference "J2")
+					(reference "Motor2")
 					(unit 1)
 				)

Commit message: s
Parts:
- renumbered U2 to M2
Changed lines of the file:
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@@
 		(dnp no)
 		(fields_autoplaced yes)
-		(property "Reference" "U2"
+		(property "Reference" "M2"
 			(at 129.1433 88.9 0)
 			(effects
@@
 			(project "Projet_Robot"
 				(path "/21a14c86-6900-4d4b-9d91-6c59051d0f41/1388fddc-2e50-4e98-ba2d-1c17e87787d8"
-					(reference "U3")
+					(reference "M1")
 					(unit 1)
 				)
 				(path "/21a14c86-6900-4d4b-9d91-6c59051d0f41/aa5a4c0f-7d13-4543-a78f-f39351de5880"
-					(reference "U2")
+					(reference "M2")
 					(unit 1)
 				)

Commit message: s
Parts:
- C22, C25: value 1 uF -> 100n; footprint Capacitor_SMD:C_0201_0603Metric -> Capacitor_SMD:C_0402_1005Metric
- R15: value 1 k -> 1k
- R16: value 4.7 k -> 4k7
Changed lines of the file:
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@@
 			)
 		)
-		(property "Value" "1 uF"
+		(property "Value" "100n"
 			(at 114.3 69.8562 0)
 			(effects
@@
 			)
 		)
-		(property "Footprint" "Capacitor_SMD:C_0201_0603Metric"
+		(property "Footprint" "Capacitor_SMD:C_0402_1005Metric"
 			(at 111.76 68.58 0)
 			(effects
@@
 			)
 		)
-		(property "Value" "1 k"
+		(property "Value" "1k"
 			(at 102.87 72.3899 0)
 			(effects
@@
 			)
 		)
-		(property "Value" "1 uF"
+		(property "Value" "100n"
 			(at 140.97 67.3035 0)
 			(effects
@@
 			)
 		)
-		(property "Footprint" "Capacitor_SMD:C_0201_0603Metric"
+		(property "Footprint" "Capacitor_SMD:C_0402_1005Metric"
 			(at 138.43 66.04 0)
 			(effects
@@
 			)
 		)
-		(property "Value" "4.7 k"
+		(property "Value" "4k7"
 			(at 93.726 83.058 0)
 			(effects
