File: Hardware/KiCad/moteur1.kicad_sch (KiCad schematic)
At the start: 8 parts, among them M2 ZXBM5210-SP

Commit message: check LF
Parts:
- removed R15: 1k, Resistor_SMD:R_0603_1608Metric, symbol Device:R_Small
- removed R16: 4k7, Resistor_SMD:R_0603_1608Metric, symbol Device:R_Small
Connections:
- net +VBAT: now also M2.6 (VREF)

Commit message: gerbers
Changed lines of the file:
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@@
 		(on_board yes)
 		(dnp no)
-		(fields_autoplaced yes)
 		(property "Reference" "TP3"
-			(at 106.68 93.2179 0)
+			(at 104.14 92.202 0)
 			(effects
 				(font
-					(size 1.27 1.27)
+					(size 1.016 1.016)
 				)
 				(justify left)
