File: Hardware/Projet_Robot/capteur.kicad_sch (KiCad schematic)
At the start: 11 parts, among them IC1 ADXL343BCCZ-RL, J1 Conn_01x05, J3 Conn_01x06, J4 Conn_01x06, J5 Conn_01x05, J6 Conn_01x06, J7 Conn_01x06

Commit message: review pcb
Parts:
- removed C26: 1u, symbol Device:C_Small
- removed J1: Conn_01x05, symbol Connector_Generic:Conn_01x05
- added J2: Conn_01x04, Connector_JST:JST_XH_B4B-XH-AM_1x04_P2.50mm_Vertical, symbol Connector_Generic:Conn_01x04
Connections:
- net TOF2_XSHUT is gone; now on net XSHUT: J4.6 (Pin_6)
- net TOF3_XSHUT is gone; now on net XSHUT: J6.6 (Pin_6)
- net TOF4_XSHUT is gone; now on net XSHUT: J7.6 (Pin_6)
- net tof1_GPIO is gone; now on net GPIO: J3.4 (Pin_4)
- net tof2_GPIO is gone; now on net GPIO: J4.4 (Pin_4)
- net tof3_GPIO is gone; now on net GPIO: J6.4 (Pin_4)
- net tof4_GPIO is gone; now on net GPIO: J7.4 (Pin_4)
- net +5V: now also J2.1 (Pin_1)
- net GND: now also J2.3 (Pin_3)
- net LIDAR_USART2_RX: now also J2.2 (Pin_2)
- net M_CTR: now also J2.4 (Pin_4)
- net ACC_INT1 renamed GPIO
- net ACC_INT2: no longer names the net of IC1.9 (INT2)
- net TOF1_XSHUT renamed XSHUT
Other:
- note added: "Capteur TOF 1"
- note removed: "Capteurs TOF"
