File: Hardware/Projet_Robot/driver_moteur.kicad_sch (KiCad schematic)
At the start: 8 parts, among them J2 Conn_01x06, U2 ZXBM5210-SP

Commit message: review pcb
Parts:
- removed J2: Conn_01x06, Connector_JST:JST_XH_S6B-XH-A_1x06_P2.50mm_Horizontal, symbol Connector_Generic:Conn_01x06
- removed TP3, TP4: TestPoint, TestPoint:TestPoint_Pad_D1.5mm, symbol Connector:TestPoint
- added J9: Conn_01x06, symbol Connector_Generic:Conn_01x06
- C23: renamed from C22; value 1 uF -> 1u
- C24: renamed from C25; value 1 uF -> 1u
- R18: renamed from R15; value 1 k -> 1k
- R19: renamed from R16; value 4.7 k -> 4k7
- renumbered U2 to U3
Connections:
- net GND: now also J9.2 (Pin_2)
- net Motor1+ renamed Mot_Out1
- net Mot_Out1: now also J9.1 (Pin_1)
- net Motor1- renamed Mot_Out2
- net Mot_Out2: now also J9.6 (Pin_6)
- net PWM_Mot1_CH1 renamed Mot_FWD
- net PWM_Mot1_CH2 renamed Mot_REV
- new net +5V: J9.5 (Pin_5)
- new net Enc_A1: J9.3 (Pin_3)
- new net Enc_B1: J9.4 (Pin_4)
Other:
- moved on the sheet: C23, C24, R18, R19, U3
