File: Hardware/Projet_Robot/regulateurs.kicad_sch (KiCad schematic)
At the start: 22 parts, among them IC2 MP1475DJ-LF-P, J8 Conn_01x02, SW2 Wurth 472121020311

Commit message: review pcb
Parts:
- C14, C18, C20: value 22u -> 22uF
- C15, C16: value 0.1u -> 0.1uF
- L2: value 4.7u -> 4.7uH
- R10: value 20 -> 20R
- R12: value 7K68 -> R_Small
- R8: value 100K -> R_Small
