File: Hardware/Projet_Robot/µcontrolleur.kicad_sch (KiCad schematic)
At the start: 27 parts, among them J11 Conn_ST_STDC14, SW1 SW_Push, SW3 SW_Push, U1 STM32G431CBUx, Y1 16MHz

Commit message: review pcb
Parts:
- removed D3, D4, D5: LED_Small, LED_SMD:LED_0603_1608Metric, symbol Device:LED_Small
- removed J11: Conn_ST_STDC14, symbol Connector:Conn_ST_STDC14
- removed R14: 1k6, Resistor_SMD:R_0603_1608Metric, symbol Device:R
- removed R5, R6: 1k, Resistor_SMD:R_0603_1608Metric, symbol Device:R
- removed SW3: SW_Push, symbol Switch:SW_Push
- added J1: Conn_02x07_Odd_Even, Connector_PinHeader_1.27mm:PinHeader_2x07_P1.27mm_Vertical_SMD, symbol Connector_Generic:Conn_02x07_Odd_Even
- added JP1, JP2: SolderJumper_2_Open, Jumper:SolderJumper-2_P1.3mm_Open_TrianglePad1.0x1.5mm, symbol Jumper:SolderJumper_2_Open
- C2: value 4u7 -> 4.7uF
- D1, D2: footprint LED_SMD:LED_0603_1608Metric -> LED_SMD:LED_0201_0603Metric
- R3: value 1k -> 100k
- R4: value 600 -> 100k
Connections:
- net +3.3V: now also J1.3 (Pin_3)
- net GND: now also J1.11 (Pin_11), J1.5 (Pin_5), J1.7 (Pin_7)
- net NRST: now also J1.12 (Pin_12)
- net SWCLK: now also J1.6 (Pin_6)
- net SWDIO: now also J1.4 (Pin_4)
- net VCP_RX: now also JP1.1 (A)
- net VCP_TX: now also JP2.2 (B)
- net ACC_INT1: no longer names the net of U1.18 (PB1)
- net ACC_INT2: no longer names the net of U1.19 (PB2)
- net BOUTON_Chat/Souris: no longer names the net of U1.29 (PC6)
- net ENC1_PH1: no longer names the net of U1.33 (PA11)
- net ENC1_PH2: no longer names the net of U1.34 (PA12)
- net ENC2_PH1: no longer names the net of U1.12 (PA4)
- net ENC2_PH2 renamed STATUS_LED
- net STATUS_LED: now also D2.2 (A)
- net LIDAR_USART2_TX: no longer names the net of U1.10 (PA2)
- net PWM_Mot1_CH1 renamed TIM1_CH1
- net PWM_Mot1_CH2 renamed TIM1_CH2
- net PWM_Mot2_CH1 renamed TIM2_CH1
- net PWM_Mot2_CH2 renamed TIM2_CH2
- net STATUS_CHAT_LED: no longer names the net of U1.4 (PC15)
- net STATUS_CHAT_LED: no longer D2.2 (A)
- net STATUS_SOURIS_LED: no longer names the net of U1.3 (PC14)
- net TOF1_XSHUT: no longer names the net of U1.25 (PB12)
- net TOF2_XSHUT: no longer names the net of U1.26 (PB13)
- net TOF3_XSHUT: no longer names the net of U1.27 (PB14)
- net TOF4_XSHUT: no longer names the net of U1.28 (PB15)
- net tof1_GPIO renamed SWO
- net SWO: now also J1.8 (Pin_8)
- net tof2_GPIO: no longer names the net of U1.42 (PB4)
- net tof3_GPIO: no longer names the net of U1.43 (PB5)
- net tof4_GPIO: no longer names the net of U1.44 (PB6)
- new net: J1.14 (Pin_14), JP2.1 (A)
- new net: J1.13 (Pin_13), JP1.2 (B)
- no-connect marks 10 -> 27
Other:
- note removed: "Bouton Chat/Souris"
- moved on the sheet: C3, C4, D1, D2, R3, R4, SW1, Y1
